File: Brewnode_PCB/ADC.sch (KiCad schematic (older format))
At the start: 7 parts

Commit message: More PCB Work
Parts:
- added JP? (x8): Jumper_2_Open, Connector_PinHeader_2.54mm:PinHeader_1x02_P2.54mm_Vertical, symbol Jumper:Jumper_2_Open
- added R? (x8): R, symbol Device:R
Connections:
- net AIN0: now also JP?.2 (B), R?.1, R?.2; no longer J?.2 (Pin_2)
- net AIN1: now also JP?.2 (B), R?.1, R?.2; no longer J?.2 (Pin_2)
- net AIN2: now also JP?.2 (B), R?.1, R?.2; no longer J?.2 (Pin_2)
- net AIN3: now also JP?.2 (B), R?.1, R?.2; no longer J?.2 (Pin_2)
- net GND: now also JP?.2 (B), JP?.2 (B), JP?.2 (B), JP?.2 (B)
- new net: JP?.1 (A), R?.2 (x4)
- new net IN_AIN0: J?.2 (Pin_2), JP?.1 (A), R?.1
- new net IN_AIN1: J?.2 (Pin_2), JP?.1 (A), R?.1
- new net IN_AIN2: J?.2 (Pin_2), JP?.1 (A), R?.1
- new net IN_AIN3: J?.2 (Pin_2), JP?.1 (A), R?.1
Other:
- note added: "0-10V"
- note added: "0-5V"
