File: Brewnode_PCB/ADC.sch (KiCad schematic (older format))
At the start: 23 parts

Commit message: More PCB Sch work
Parts:
- gave numbers to parts that had none: 23
Changed lines of the file:
@@
 $EndDescr
 $Comp
-L Analog_ADC:ADS1115IDGS U?
+L Analog_ADC:ADS1115IDGS U2
 U 1 1 5F671F24
 P 6000 3000
-F 0 "U?" H 6000 3681 50  0000 C CNN
+F 0 "U2" H 6000 3681 50  0000 C CNN
 F 1 "ADS1115IDGS" H 6000 3590 50  0000 C CNN
 F 2 "Package_SO:TSSOP-10_3x3mm_P0.5mm" H 6000 2500 50  0001 C CNN
@@
 $EndComp
 $Comp
-L power:+5V #PWR?
+L power:+5V #PWR021
 U 1 1 5F672F0A
 P 5700 2100
-F 0 "#PWR?" H 5700 1950 50  0001 C CNN
+F 0 "#PWR021" H 5700 1950 50  0001 C CNN
 F 1 "+5V" H 5715 2273 50  0000 C CNN
 F 2 "" H 5700 2100 50  0001 C CNN
@@
 $EndComp
 $Comp
-L power:GND #PWR?
+L power:GND #PWR022
 U 1 1 5F6733C6
 P 5700 3500
-F 0 "#PWR?" H 5700 3250 50  0001 C CNN
+F 0 "#PWR022" H 5700 3250 50  0001 C CNN
 F 1 "GND" H 5705 3327 50  0000 C CNN
 F 2 "" H 5700 3500 50  0001 C CNN
@@
 $EndComp
 $Comp
-L Connector:Screw_Terminal_01x03 J?
+L Connector:Screw_Terminal_01x03 J9
 U 1 1 5F67AE54
 P 8950 2150
-F 0 "J?" H 9030 2192 50  0000 L CNN
+F 0 "J9" H 9030 2192 50  0000 L CNN
 F 1 "Screw_Terminal_01x03" H 9030 2101 50  0000 L CNN
 F 2 "" H 8950 2150 50  0001 C CNN
@@
 $EndComp
 $Comp
-L Connector:Screw_Terminal_01x03 J?
+L Connector:Screw_Terminal_01x03 J10
 U 1 1 5F67CFB3
 P 8950 2650
-F 0 "J?" H 9030 2692 50  0000 L CNN
+F 0 "J10" H 9030 2692 50  0000 L CNN
 F 1 "Screw_Terminal_01x03" H 9030 2601 50  0000 L CNN
 F 2 "" H 8950 2650 50  0001 C CNN
@@
 $EndComp
 $Comp
-L Connector:Screw_Terminal_01x03 J?
+L Connector:Screw_Terminal_01x03 J11
 U 1 1 5F67D7CC
 P 8950 3150
-F 0 "J?" H 9030 3192 50  0000 L CNN
+F 0 "J11" H 9030 3192 50  0000 L CNN
 F 1 "Screw_Terminal_01x03" H 9030 3101 50  0000 L CNN
 F 2 "" H 8950 3150 50  0001 C CNN
@@
 $EndComp
 $Comp
-L Connector:Screw_Terminal_01x03 J?
+L Connector:Screw_Terminal_01x03 J12
 U 1 1 5F67DB58
 P 8950 3650
-F 0 "J?" H 9030 3692 50  0000 L CNN
+F 0 "J12" H 9030 3692 50  0000 L CNN
 F 1 "Screw_Terminal_01x03" H 9030 3601 50  0000 L CNN
 F 2 "" H 8950 3650 50  0001 C CNN
@@
 $EndComp
 $Comp
-L power:+5V #PWR?
+L power:+5V #PWR026
 U 1 1 5F68337D
 P 8500 1600
-F 0 "#PWR?" H 8500 1450 50  0001 C CNN
+F 0 "#PWR026" H 8500 1450 50  0001 C CNN
 F 1 "+5V" H 8515 1773 50  0000 C CNN
 F 2 "" H 8500 1600 50  0001 C CNN
@@
 $EndComp
 $Comp
-L power:GND #PWR?
+L power:GND #PWR025
 U 1 1 5F683A9D
 P 8400 3900
-F 0 "#PWR?" H 8400 3650 50  0001 C CNN
+F 0 "#PWR025" H 8400 3650 50  0001 C CNN
 F 1 "GND" H 8405 3727 50  0000 C CNN
 F 2 "" H 8400 3900 50  0001 C CNN
@@
 	6400 2800 6600 2800
 $Comp
-L Device:C C?
+L Device:C C4
 U 1 1 5F692BD5
 P 4550 2850
-F 0 "C?" H 4665 2896 50  0000 L CNN
+F 0 "C4" H 4665 2896 50  0000 L CNN
 F 1 "C" H 4665 2805 50  0000 L CNN
 F 2 "" H 4588 2700 50  0001 C CNN
@@
 AIN3
 $Comp
-L Device:CP C?
+L Device:CP C5
 U 1 1 5F69915C
 P 7500 2850
-F 0 "C?" H 7618 2896 50  0000 L CNN
+F 0 "C5" H 7618 2896 50  0000 L CNN
 F 1 "CP" H 7618 2805 50  0000 L CNN
 F 2 "" H 7538 2700 50  0001 C CNN
@@
 IN_AIN3
 $Comp
-L Device:R R?
+L Device:R R8
 U 1 1 5F6380A2
 P 850 5600
-F 0 "R?" H 920 5646 50  0000 L CNN
+F 0 "R8" H 920 5646 50  0000 L CNN
 F 1 "R" H 920 5555 50  0000 L CNN
 F 2 "" V 780 5600 50  0001 C CNN
@@
 $EndComp
 $Comp
-L Device:R R?
+L Device:R R7
 U 1 1 5F6380A8
 P 850 5000
-F 0 "R?" H 920 5046 50  0000 L CNN
+F 0 "R7" H 920 5046 50  0000 L CNN
 F 1 "R" H 920 4955 50  0000 L CNN
 F 2 "" V 780 5000 50  0001 C CNN
@@
 	850  4700 1350 4700
 $Comp
-L power:GND #PWR?
+L power:GND #PWR019
 U 1 1 5F6380BC
 P 2000 5950
-F 0 "#PWR?" H 2000 5700 50  0001 C CNN
+F 0 "#PWR019" H 2000 5700 50  0001 C CNN
 F 1 "GND" H 2005 5777 50  0000 C CNN
 F 2 "" H 2000 5950 50  0001 C CNN
@@
 IN_AIN0
 $Comp
-L Jumper:Jumper_2_Open JP?
+L Jumper:Jumper_2_Open JP2
 U 1 1 5F64E0CE
 P 1750 5800
-F 0 "JP?" H 1750 6035 50  0000 C CNN
+F 0 "JP2" H 1750 6035 50  0000 C CNN
 F 1 "Jumper_2_Open" H 1750 5944 50  0000 C CNN
 F 2 "Connector_PinHeader_2.54mm:PinHeader_1x02_P2.54mm_Vertical" H 1750 5800 50  0001 C CNN
@@
 $EndComp
 $Comp
-L Jumper:Jumper_2_Open JP?
+L Jumper:Jumper_2_Open JP1
 U 1 1 5F64EF25
 P 1750 5000
-F 0 "JP?" H 1750 5235 50  0000 C CNN
+F 0 "JP1" H 1750 5235 50  0000 C CNN
 F 1 "Jumper_2_Open" H 1750 5144 50  0000 C CNN
 F 2 "Connector_PinHeader_2.54mm:PinHeader_1x02_P2.54mm_Vertical" H 1750 5000 50  0001 C CNN
@@
 0-10V
 $Comp
-L Device:R R?
+L Device:R R10
 U 1 1 5F6912D6
 P 2850 5600
-F 0 "R?" H 2920 5646 50  0000 L CNN
+F 0 "R10" H 2920 5646 50  0000 L CNN
 F 1 "R" H 2920 5555 50  0000 L CNN
 F 2 "" V 2780 5600 50  0001 C CNN
@@
 $EndComp
 $Comp
-L Device:R R?
+L Device:R R9
 U 1 1 5F6912DC
 P 2850 5000
-F 0 "R?" H 2920 5046 50  0000 L CNN
+F 0 "R9" H 2920 5046 50  0000 L CNN
 F 1 "R" H 2920 4955 50  0000 L CNN
 F 2 "" V 2780 5000 50  0001 C CNN
@@
 	2850 4700 3350 4700
 $Comp
-L power:GND #PWR?
+L power:GND #PWR020
 U 1 1 5F6912E4
 P 4000 5950
-F 0 "#PWR?" H 4000 5700 50  0001 C CNN
+F 0 "#PWR020" H 4000 5700 50  0001 C CNN
 F 1 "GND" H 4005 5777 50  0000 C CNN
 F 2 "" H 4000 5950 50  0001 C CNN
@@
 IN_AIN1
 $Comp
-L Jumper:Jumper_2_Open JP?
+L Jumper:Jumper_2_Open JP4
 U 1 1 5F6912EC
 P 3750 5800
-F 0 "JP?" H 3750 6035 50  0000 C CNN
+F 0 "JP4" H 3750 6035 50  0000 C CNN
 F 1 "Jumper_2_Open" H 3750 5944 50  0000 C CNN
 F 2 "Connector_PinHeader_2.54mm:PinHeader_1x02_P2.54mm_Vertical" H 3750 5800 50  0001 C CNN
@@
 $EndComp
 $Comp
-L Jumper:Jumper_2_Open JP?
+L Jumper:Jumper_2_Open JP3
 U 1 1 5F6912F2
 P 3750 5000
-F 0 "JP?" H 3750 5235 50  0000 C CNN
+F 0 "JP3" H 3750 5235 50  0000 C CNN
 F 1 "Jumper_2_Open" H 3750 5144 50  0000 C CNN
 F 2 "Connector_PinHeader_2.54mm:PinHeader_1x02_P2.54mm_Vertical" H 3750 5000 50  0001 C CNN
@@
 0-10V
 $Comp
-L Device:R R?
+L Device:R R12
 U 1 1 5F694267
 P 4850 5600
-F 0 "R?" H 4920 5646 50  0000 L CNN
+F 0 "R12" H 4920 5646 50  0000 L CNN
 F 1 "R" H 4920 5555 50  0000 L CNN
 F 2 "" V 4780 5600 50  0001 C CNN
@@
 $EndComp
 $Comp
-L Device:R R?
+L Device:R R11
 U 1 1 5F69426D
 P 4850 5000
-F 0 "R?" H 4920 5046 50  0000 L CNN
+F 0 "R11" H 4920 5046 50  0000 L CNN
 F 1 "R" H 4920 4955 50  0000 L CNN
 F 2 "" V 4780 5000 50  0001 C CNN
@@
 	4850 4700 5350 4700
 $Comp
-L power:GND #PWR?
+L power:GND #PWR023
 U 1 1 5F694275
 P 6000 5950
-F 0 "#PWR?" H 6000 5700 50  0001 C CNN
+F 0 "#PWR023" H 6000 5700 50  0001 C CNN
 F 1 "GND" H 6005 5777 50  0000 C CNN
 F 2 "" H 6000 5950 50  0001 C CNN
@@
 IN_AIN2
 $Comp
-L Jumper:Jumper_2_Open JP?
+L Jumper:Jumper_2_Open JP6
 U 1 1 5F69427D
 P 5750 5800
-F 0 "JP?" H 5750 6035 50  0000 C CNN
+F 0 "JP6" H 5750 6035 50  0000 C CNN
 F 1 "Jumper_2_Open" H 5750 5944 50  0000 C CNN
 F 2 "Connector_PinHeader_2.54mm:PinHeader_1x02_P2.54mm_Vertical" H 5750 5800 50  0001 C CNN
@@
 $EndComp
 $Comp
-L Jumper:Jumper_2_Open JP?
+L Jumper:Jumper_2_Open JP5
 U 1 1 5F694283
 P 5750 5000
-F 0 "JP?" H 5750 5235 50  0000 C CNN
+F 0 "JP5" H 5750 5235 50  0000 C CNN
 F 1 "Jumper_2_Open" H 5750 5144 50  0000 C CNN
 F 2 "Connector_PinHeader_2.54mm:PinHeader_1x02_P2.54mm_Vertical" H 5750 5000 50  0001 C CNN
@@
 0-10V
 $Comp
-L Device:R R?
+L Device:R R14
 U 1 1 5F6C52F3
 P 6850 5600
-F 0 "R?" H 6920 5646 50  0000 L CNN
+F 0 "R14" H 6920 5646 50  0000 L CNN
 F 1 "R" H 6920 5555 50  0000 L CNN
 F 2 "" V 6780 5600 50  0001 C CNN
@@
 $EndComp
 $Comp
-L Device:R R?
+L Device:R R13
 U 1 1 5F6C52F9
 P 6850 5000
-F 0 "R?" H 6920 5046 50  0000 L CNN
+F 0 "R13" H 6920 5046 50  0000 L CNN
 F 1 "R" H 6920 4955 50  0000 L CNN
 F 2 "" V 6780 5000 50  0001 C CNN
@@
 	6850 4700 7350 4700
 $Comp
-L power:GND #PWR?
+L power:GND #PWR024
 U 1 1 5F6C5301
 P 8000 5950
-F 0 "#PWR?" H 8000 5700 50  0001 C CNN
+F 0 "#PWR024" H 8000 5700 50  0001 C CNN
 F 1 "GND" H 8005 5777 50  0000 C CNN
 F 2 "" H 8000 5950 50  0001 C CNN
@@
 IN_AIN3
 $Comp
-L Jumper:Jumper_2_Open JP?
+L Jumper:Jumper_2_Open JP8
 U 1 1 5F6C5309
 P 7750 5800
-F 0 "JP?" H 7750 6035 50  0000 C CNN
+F 0 "JP8" H 7750 6035 50  0000 C CNN
 F 1 "Jumper_2_Open" H 7750 5944 50  0000 C CNN
 F 2 "Connector_PinHeader_2.54mm:PinHeader_1x02_P2.54mm_Vertical" H 7750 5800 50  0001 C CNN
@@
 $EndComp
 $Comp
-L Jumper:Jumper_2_Open JP?
+L Jumper:Jumper_2_Open JP7
 U 1 1 5F6C530F
 P 7750 5000
-F 0 "JP?" H 7750 5235 50  0000 C CNN
+F 0 "JP7" H 7750 5235 50  0000 C CNN
 F 1 "Jumper_2_Open" H 7750 5144 50  0000 C CNN
 F 2 "Connector_PinHeader_2.54mm:PinHeader_1x02_P2.54mm_Vertical" H 7750 5000 50  0001 C CNN

Commit message: More PCB Sch work
Parts:
- C4: value C -> 100nF; footprint (none) -> Capacitor_SMD:C_0402_1005Metric; LCSC (none) -> C1525; Mfc (none) -> CL05B104KO5NNNC
- C5: value CP -> 47uF; footprint (none) -> Capacitor_SMD:CP_Elec_6.3x5.3; LCSC (none) -> C249778; Mfc (none) -> VEZ470M1CTR-0605
- J10, J11, J12, J9: LCSC (none) -> C8377; Mfc (none) -> WJ2EDGRC-5.08-3P
- R10, R11, R12, R13, R14, R7, R8, R9: value R -> 8.2kOhm; LCSC (none) -> C407435; Mfc (none) -> 0805W8D8201T5E
- U2: LCSC (none) -> C37593; Mfc (none) -> ADS1115IDGSR
Changed lines of the file:
@@
 F 1 "ADS1115IDGS" H 6000 3590 50  0000 C CNN
 F 2 "Package_SO:TSSOP-10_3x3mm_P0.5mm" H 6000 2500 50  0001 C CNN
-F 3 "http://www.ti.com/lit/ds/symlink/ads1113.pdf" H 5950 2100 50  0001 C CNN
+F 3 "https://datasheet.lcsc.com/szlcsc/1809192322_Texas-Instruments-ADS1115IDGSR_C37593.pdf" H 5950 2100 50  0001 C CNN
+F 4 "C37593" H 6000 3000 50  0001 C CNN "LCSC"
+F 5 "ADS1115IDGSR" H 6000 3000 50  0001 C CNN "Mfc"
 	1    6000 3000
 	1    0    0    -1
@@
 F 1 "Screw_Terminal_01x03" H 9030 2101 50  0000 L CNN
 F 2 "" H 8950 2150 50  0001 C CNN
-F 3 "~" H 8950 2150 50  0001 C CNN
+F 3 "https://datasheet.lcsc.com/szlcsc/1912251632_Ningbo-Kangnex-Elec-WJ2EDGRC-5-08-3P_C8377.pdf" H 8950 2150 50  0001 C CNN
+F 4 "C8377" H 8950 2150 50  0001 C CNN "LCSC"
+F 5 "WJ2EDGRC-5.08-3P" H 8950 2150 50  0001 C CNN "Mfc"
 	1    8950 2150
 	1    0    0    -1
@@
 F 1 "Screw_Terminal_01x03" H 9030 2601 50  0000 L CNN
 F 2 "" H 8950 2650 50  0001 C CNN
-F 3 "~" H 8950 2650 50  0001 C CNN
+F 3 "https://datasheet.lcsc.com/szlcsc/1912251632_Ningbo-Kangnex-Elec-WJ2EDGRC-5-08-3P_C8377.pdf" H 8950 2650 50  0001 C CNN
+F 4 "C8377" H 8950 2650 50  0001 C CNN "LCSC"
+F 5 "WJ2EDGRC-5.08-3P" H 8950 2650 50  0001 C CNN "Mfc"
 	1    8950 2650
 	1    0    0    -1
@@
 F 1 "Screw_Terminal_01x03" H 9030 3101 50  0000 L CNN
 F 2 "" H 8950 3150 50  0001 C CNN
-F 3 "~" H 8950 3150 50  0001 C CNN
+F 3 "https://datasheet.lcsc.com/szlcsc/1912251632_Ningbo-Kangnex-Elec-WJ2EDGRC-5-08-3P_C8377.pdf" H 8950 3150 50  0001 C CNN
+F 4 "C8377" H 8950 3150 50  0001 C CNN "LCSC"
+F 5 "WJ2EDGRC-5.08-3P" H 8950 3150 50  0001 C CNN "Mfc"
 	1    8950 3150
 	1    0    0    -1
@@
 F 1 "Screw_Terminal_01x03" H 9030 3601 50  0000 L CNN
 F 2 "" H 8950 3650 50  0001 C CNN
-F 3 "~" H 8950 3650 50  0001 C CNN
+F 3 "https://datasheet.lcsc.com/szlcsc/1912251632_Ningbo-Kangnex-Elec-WJ2EDGRC-5-08-3P_C8377.pdf" H 8950 3650 50  0001 C CNN
+F 4 "C8377" H 8950 3650 50  0001 C CNN "LCSC"
+F 5 "WJ2EDGRC-5.08-3P" H 8950 3650 50  0001 C CNN "Mfc"
 	1    8950 3650
 	1    0    0    -1
@@
 Wire Wire Line
 	5700 3500 5700 3450
-Wire Wire Line
-	5700 3450 6000 3450
-Wire Wire Line
-	6000 3450 6000 3400
 Text HLabel 6600 3000 2    50   BiDi ~ 0
 5V_ADC_SCL
@@
 	6500 3200 6500 3450
 Wire Wire Line
-	6500 3450 6000 3450
-Connection ~ 6000 3450
-Wire Wire Line
 	6400 3000 6600 3000
 Wire Wire Line
@@
 P 4550 2850
 F 0 "C4" H 4665 2896 50  0000 L CNN
-F 1 "C" H 4665 2805 50  0000 L CNN
-F 2 "" H 4588 2700 50  0001 C CNN
-F 3 "~" H 4550 2850 50  0001 C CNN
+F 1 "100nF" H 4665 2805 50  0000 L CNN
+F 2 "Capacitor_SMD:C_0402_1005Metric" H 4588 2700 50  0001 C CNN
+F 3 "https://datasheet.lcsc.com/szlcsc/1810191219_Samsung-Electro-Mechanics-CL05B104KO5NNNC_C1525.pdf" H 4550 2850 50  0001 C CNN
+F 4 "C1525" H 4550 2850 50  0001 C CNN "LCSC"
+F 5 "CL05B104KO5NNNC" H 4550 2850 50  0001 C CNN "Mfc"
 	1    4550 2850
 	1    0    0    -1
@@
 Wire Wire Line
 	4550 3450 5700 3450
-Connection ~ 5700 3450
 Wire Wire Line
 	5600 3000 5200 3000
@@
 P 7500 2850
 F 0 "C5" H 7618 2896 50  0000 L CNN
-F 1 "CP" H 7618 2805 50  0000 L CNN
-F 2 "" H 7538 2700 50  0001 C CNN
-F 3 "~" H 7500 2850 50  0001 C CNN
+F 1 "47uF" H 7618 2805 50  0000 L CNN
+F 2 "Capacitor_SMD:CP_Elec_6.3x5.3" H 7538 2700 50  0001 C CNN
+F 3 "https://datasheet.lcsc.com/szlcsc/1912111437_Lelon-VEZ470M1CTR-0605_C249778.pdf" H 7500 2850 50  0001 C CNN
+F 4 "C249778" H 7500 2850 50  0001 C CNN "LCSC"
+F 5 "	VEZ470M1CTR-0605" H 7500 2850 50  0001 C CNN "Mfc"
 	1    7500 2850
 	1    0    0    -1
@@
 P 850 5600
 F 0 "R8" H 920 5646 50  0000 L CNN
-F 1 "R" H 920 5555 50  0000 L CNN
+F 1 "8.2kOhm" H 920 5555 50  0000 L CNN
 F 2 "" V 780 5600 50  0001 C CNN
-F 3 "~" H 850 5600 50  0001 C CNN
+F 3 "https://datasheet.lcsc.com/szlcsc/1912111437_UNI-ROYAL-Uniroyal-Elec-0805W8D8201T5E_C407435.pdf" H 850 5600 50  0001 C CNN
+F 4 "C407435" H 850 5600 50  0001 C CNN "LCSC"
+F 5 "0805W8D8201T5E" H 850 5600 50  0001 C CNN "Mfc"
 	1    850  5600
 	1    0    0    -1
@@
 P 850 5000
 F 0 "R7" H 920 5046 50  0000 L CNN
-F 1 "R" H 920 4955 50  0000 L CNN
+F 1 "8.2kOhm" H 920 4955 50  0000 L CNN
 F 2 "" V 780 5000 50  0001 C CNN
-F 3 "~" H 850 5000 50  0001 C CNN
+F 3 "https://datasheet.lcsc.com/szlcsc/1912111437_UNI-ROYAL-Uniroyal-Elec-0805W8D8201T5E_C407435.pdf" H 850 5000 50  0001 C CNN
+F 4 "C407435" H 850 5000 50  0001 C CNN "LCSC"
+F 5 "0805W8D8201T5E" H 850 5000 50  0001 C CNN "Mfc"
 	1    850  5000
 	1    0    0    -1
@@
 P 2850 5600
 F 0 "R10" H 2920 5646 50  0000 L CNN
-F 1 "R" H 2920 5555 50  0000 L CNN
+F 1 "8.2kOhm" H 2920 5555 50  0000 L CNN
 F 2 "" V 2780 5600 50  0001 C CNN
-F 3 "~" H 2850 5600 50  0001 C CNN
+F 3 "https://datasheet.lcsc.com/szlcsc/1912111437_UNI-ROYAL-Uniroyal-Elec-0805W8D8201T5E_C407435.pdf" H 2850 5600 50  0001 C CNN
+F 4 "C407435" H 2850 5600 50  0001 C CNN "LCSC"
+F 5 "0805W8D8201T5E" H 2850 5600 50  0001 C CNN "Mfc"
 	1    2850 5600
 	1    0    0    -1
@@
 P 2850 5000
 F 0 "R9" H 2920 5046 50  0000 L CNN
-F 1 "R" H 2920 4955 50  0000 L CNN
+F 1 "8.2kOhm" H 2920 4955 50  0000 L CNN
 F 2 "" V 2780 5000 50  0001 C CNN
-F 3 "~" H 2850 5000 50  0001 C CNN
+F 3 "https://datasheet.lcsc.com/szlcsc/1912111437_UNI-ROYAL-Uniroyal-Elec-0805W8D8201T5E_C407435.pdf" H 2850 5000 50  0001 C CNN
+F 4 "C407435" H 2850 5000 50  0001 C CNN "LCSC"
+F 5 "0805W8D8201T5E" H 2850 5000 50  0001 C CNN "Mfc"
 	1    2850 5000
 	1    0    0    -1
@@
 P 4850 5600
 F 0 "R12" H 4920 5646 50  0000 L CNN
-F 1 "R" H 4920 5555 50  0000 L CNN
+F 1 "8.2kOhm" H 4920 5555 50  0000 L CNN
 F 2 "" V 4780 5600 50  0001 C CNN
-F 3 "~" H 4850 5600 50  0001 C CNN
+F 3 "https://datasheet.lcsc.com/szlcsc/1912111437_UNI-ROYAL-Uniroyal-Elec-0805W8D8201T5E_C407435.pdf" H 4850 5600 50  0001 C CNN
+F 4 "C407435" H 4850 5600 50  0001 C CNN "LCSC"
+F 5 "0805W8D8201T5E" H 4850 5600 50  0001 C CNN "Mfc"
 	1    4850 5600
 	1    0    0    -1
@@
 P 4850 5000
 F 0 "R11" H 4920 5046 50  0000 L CNN
-F 1 "R" H 4920 4955 50  0000 L CNN
+F 1 "8.2kOhm" H 4920 4955 50  0000 L CNN
 F 2 "" V 4780 5000 50  0001 C CNN
-F 3 "~" H 4850 5000 50  0001 C CNN
+F 3 "https://datasheet.lcsc.com/szlcsc/1912111437_UNI-ROYAL-Uniroyal-Elec-0805W8D8201T5E_C407435.pdf" H 4850 5000 50  0001 C CNN
+F 4 "C407435" H 4850 5000 50  0001 C CNN "LCSC"
+F 5 "0805W8D8201T5E" H 4850 5000 50  0001 C CNN "Mfc"
 	1    4850 5000
 	1    0    0    -1
@@
 P 6850 5600
 F 0 "R14" H 6920 5646 50  0000 L CNN
-F 1 "R" H 6920 5555 50  0000 L CNN
+F 1 "8.2kOhm" H 6920 5555 50  0000 L CNN
 F 2 "" V 6780 5600 50  0001 C CNN
-F 3 "~" H 6850 5600 50  0001 C CNN
+F 3 "https://datasheet.lcsc.com/szlcsc/1912111437_UNI-ROYAL-Uniroyal-Elec-0805W8D8201T5E_C407435.pdf" H 6850 5600 50  0001 C CNN
+F 4 "C407435" H 6850 5600 50  0001 C CNN "LCSC"
+F 5 "0805W8D8201T5E" H 6850 5600 50  0001 C CNN "Mfc"
 	1    6850 5600
 	1    0    0    -1
@@
 P 6850 5000
 F 0 "R13" H 6920 5046 50  0000 L CNN
-F 1 "R" H 6920 4955 50  0000 L CNN
+F 1 "8.2kOhm" H 6920 4955 50  0000 L CNN
 F 2 "" V 6780 5000 50  0001 C CNN
-F 3 "~" H 6850 5000 50  0001 C CNN
+F 3 "https://datasheet.lcsc.com/szlcsc/1912111437_UNI-ROYAL-Uniroyal-Elec-0805W8D8201T5E_C407435.pdf" H 6850 5000 50  0001 C CNN
+F 4 "C407435" H 6850 5000 50  0001 C CNN "LCSC"
+F 5 "0805W8D8201T5E" H 6850 5000 50  0001 C CNN "Mfc"
 	1    6850 5000
 	1    0    0    -1
@@
 Text Notes 7600 5950 0    50   ~ 0
 0-10V
+Wire Wire Line
+	5700 3450 6000 3450
+Connection ~ 5700 3450
+Wire Wire Line
+	6000 3400 6000 3450
+Connection ~ 6000 3450
+Wire Wire Line
+	6000 3450 6500 3450
 $EndSCHEMATC

Commit message: Done PCB Sch Work
Parts:
- J10, J9: footprint (none) -> Connector_Phoenix_MSTB:PhoenixContact_MSTBA_2,5_3-G-5,08_1x03_P5.08mm_Horizontal
- J11, J12: footprint (none) -> Connector_Phoenix_MSTB:PhoenixContact_MSTBVA_2,5_3-G-5,08_1x03_P5.08mm_Vertical; LCSC C8377 -> C8412; Mfc WJ2EDGRC-5.08-3P -> WJ2EDGVC-5.08-3P
- R10, R11, R12, R13, R14, R7, R8, R9: footprint (none) -> Resistor_SMD:R_0805_2012Metric_Pad1.15x1.40mm_HandSolder
- U2: footprint Package_SO:TSSOP-10_3x3mm_P0.5mm -> Package_SO:VSSOP-10_3x3mm_P0.5mm
Changed lines of the file:
@@
 F 0 "U2" H 6000 3681 50  0000 C CNN
 F 1 "ADS1115IDGS" H 6000 3590 50  0000 C CNN
-F 2 "Package_SO:TSSOP-10_3x3mm_P0.5mm" H 6000 2500 50  0001 C CNN
+F 2 "Package_SO:VSSOP-10_3x3mm_P0.5mm" H 6000 2500 50  0001 C CNN
 F 3 "https://datasheet.lcsc.com/szlcsc/1809192322_Texas-Instruments-ADS1115IDGSR_C37593.pdf" H 5950 2100 50  0001 C CNN
 F 4 "C37593" H 6000 3000 50  0001 C CNN "LCSC"
@@
 F 0 "J9" H 9030 2192 50  0000 L CNN
 F 1 "Screw_Terminal_01x03" H 9030 2101 50  0000 L CNN
-F 2 "" H 8950 2150 50  0001 C CNN
+F 2 "Connector_Phoenix_MSTB:PhoenixContact_MSTBA_2,5_3-G-5,08_1x03_P5.08mm_Horizontal" H 8950 2150 50  0001 C CNN
 F 3 "https://datasheet.lcsc.com/szlcsc/1912251632_Ningbo-Kangnex-Elec-WJ2EDGRC-5-08-3P_C8377.pdf" H 8950 2150 50  0001 C CNN
-F 4 "C8377" H 8950 2150 50  0001 C CNN "LCSC"
+F 4 "C8377" H 9250 2200 50  0000 C CNN "LCSC"
 F 5 "WJ2EDGRC-5.08-3P" H 8950 2150 50  0001 C CNN "Mfc"
 	1    8950 2150
@@
 F 0 "J10" H 9030 2692 50  0000 L CNN
 F 1 "Screw_Terminal_01x03" H 9030 2601 50  0000 L CNN
-F 2 "" H 8950 2650 50  0001 C CNN
+F 2 "Connector_Phoenix_MSTB:PhoenixContact_MSTBA_2,5_3-G-5,08_1x03_P5.08mm_Horizontal" H 8950 2650 50  0001 C CNN
 F 3 "https://datasheet.lcsc.com/szlcsc/1912251632_Ningbo-Kangnex-Elec-WJ2EDGRC-5-08-3P_C8377.pdf" H 8950 2650 50  0001 C CNN
-F 4 "C8377" H 8950 2650 50  0001 C CNN "LCSC"
+F 4 "C8377" H 9300 2700 50  0000 C CNN "LCSC"
 F 5 "WJ2EDGRC-5.08-3P" H 8950 2650 50  0001 C CNN "Mfc"
 	1    8950 2650
@@
 F 0 "J11" H 9030 3192 50  0000 L CNN
 F 1 "Screw_Terminal_01x03" H 9030 3101 50  0000 L CNN
-F 2 "" H 8950 3150 50  0001 C CNN
-F 3 "https://datasheet.lcsc.com/szlcsc/1912251632_Ningbo-Kangnex-Elec-WJ2EDGRC-5-08-3P_C8377.pdf" H 8950 3150 50  0001 C CNN
-F 4 "C8377" H 8950 3150 50  0001 C CNN "LCSC"
-F 5 "WJ2EDGRC-5.08-3P" H 8950 3150 50  0001 C CNN "Mfc"
+F 2 "Connector_Phoenix_MSTB:PhoenixContact_MSTBVA_2,5_3-G-5,08_1x03_P5.08mm_Vertical" H 8950 3150 50  0001 C CNN
+F 3 "https://datasheet.lcsc.com/szlcsc/1912251634_Ningbo-Kangnex-Elec-WJ2EDGVC-5-08-3P_C8412.pdf" H 8950 3150 50  0001 C CNN
+F 4 "C8412" H 9300 3200 50  0000 C CNN "LCSC"
+F 5 "WJ2EDGVC-5.08-3P" H 8950 3150 50  0001 C CNN "Mfc"
 	1    8950 3150
 	1    0    0    -1
@@
 F 0 "J12" H 9030 3692 50  0000 L CNN
 F 1 "Screw_Terminal_01x03" H 9030 3601 50  0000 L CNN
-F 2 "" H 8950 3650 50  0001 C CNN
-F 3 "https://datasheet.lcsc.com/szlcsc/1912251632_Ningbo-Kangnex-Elec-WJ2EDGRC-5-08-3P_C8377.pdf" H 8950 3650 50  0001 C CNN
-F 4 "C8377" H 8950 3650 50  0001 C CNN "LCSC"
-F 5 "WJ2EDGRC-5.08-3P" H 8950 3650 50  0001 C CNN "Mfc"
+F 2 "Connector_Phoenix_MSTB:PhoenixContact_MSTBVA_2,5_3-G-5,08_1x03_P5.08mm_Vertical" H 8950 3650 50  0001 C CNN
+F 3 "https://datasheet.lcsc.com/szlcsc/1912251634_Ningbo-Kangnex-Elec-WJ2EDGVC-5-08-3P_C8412.pdf" H 8950 3650 50  0001 C CNN
+F 4 "C8412" H 9300 3700 50  0000 C CNN "LCSC"
+F 5 "WJ2EDGVC-5.08-3P" H 8950 3650 50  0001 C CNN "Mfc"
 	1    8950 3650
 	1    0    0    -1
@@
 F 0 "R8" H 920 5646 50  0000 L CNN
 F 1 "8.2kOhm" H 920 5555 50  0000 L CNN
-F 2 "" V 780 5600 50  0001 C CNN
+F 2 "Resistor_SMD:R_0805_2012Metric_Pad1.15x1.40mm_HandSolder" V 780 5600 50  0001 C CNN
 F 3 "https://datasheet.lcsc.com/szlcsc/1912111437_UNI-ROYAL-Uniroyal-Elec-0805W8D8201T5E_C407435.pdf" H 850 5600 50  0001 C CNN
 F 4 "C407435" H 850 5600 50  0001 C CNN "LCSC"
@@
 F 0 "R7" H 920 5046 50  0000 L CNN
 F 1 "8.2kOhm" H 920 4955 50  0000 L CNN
-F 2 "" V 780 5000 50  0001 C CNN
+F 2 "Resistor_SMD:R_0805_2012Metric_Pad1.15x1.40mm_HandSolder" V 780 5000 50  0001 C CNN
 F 3 "https://datasheet.lcsc.com/szlcsc/1912111437_UNI-ROYAL-Uniroyal-Elec-0805W8D8201T5E_C407435.pdf" H 850 5000 50  0001 C CNN
 F 4 "C407435" H 850 5000 50  0001 C CNN "LCSC"
@@
 F 0 "R10" H 2920 5646 50  0000 L CNN
 F 1 "8.2kOhm" H 2920 5555 50  0000 L CNN
-F 2 "" V 2780 5600 50  0001 C CNN
+F 2 "Resistor_SMD:R_0805_2012Metric_Pad1.15x1.40mm_HandSolder" V 2780 5600 50  0001 C CNN
 F 3 "https://datasheet.lcsc.com/szlcsc/1912111437_UNI-ROYAL-Uniroyal-Elec-0805W8D8201T5E_C407435.pdf" H 2850 5600 50  0001 C CNN
 F 4 "C407435" H 2850 5600 50  0001 C CNN "LCSC"
@@
 F 0 "R9" H 2920 5046 50  0000 L CNN
 F 1 "8.2kOhm" H 2920 4955 50  0000 L CNN
-F 2 "" V 2780 5000 50  0001 C CNN
+F 2 "Resistor_SMD:R_0805_2012Metric_Pad1.15x1.40mm_HandSolder" V 2780 5000 50  0001 C CNN
 F 3 "https://datasheet.lcsc.com/szlcsc/1912111437_UNI-ROYAL-Uniroyal-Elec-0805W8D8201T5E_C407435.pdf" H 2850 5000 50  0001 C CNN
 F 4 "C407435" H 2850 5000 50  0001 C CNN "LCSC"
@@
 F 0 "R12" H 4920 5646 50  0000 L CNN
 F 1 "8.2kOhm" H 4920 5555 50  0000 L CNN
-F 2 "" V 4780 5600 50  0001 C CNN
+F 2 "Resistor_SMD:R_0805_2012Metric_Pad1.15x1.40mm_HandSolder" V 4780 5600 50  0001 C CNN
 F 3 "https://datasheet.lcsc.com/szlcsc/1912111437_UNI-ROYAL-Uniroyal-Elec-0805W8D8201T5E_C407435.pdf" H 4850 5600 50  0001 C CNN
 F 4 "C407435" H 4850 5600 50  0001 C CNN "LCSC"
@@
 F 0 "R11" H 4920 5046 50  0000 L CNN
 F 1 "8.2kOhm" H 4920 4955 50  0000 L CNN
-F 2 "" V 4780 5000 50  0001 C CNN
+F 2 "Resistor_SMD:R_0805_2012Metric_Pad1.15x1.40mm_HandSolder" V 4780 5000 50  0001 C CNN
 F 3 "https://datasheet.lcsc.com/szlcsc/1912111437_UNI-ROYAL-Uniroyal-Elec-0805W8D8201T5E_C407435.pdf" H 4850 5000 50  0001 C CNN
 F 4 "C407435" H 4850 5000 50  0001 C CNN "LCSC"
@@
 F 0 "R14" H 6920 5646 50  0000 L CNN
 F 1 "8.2kOhm" H 6920 5555 50  0000 L CNN
-F 2 "" V 6780 5600 50  0001 C CNN
+F 2 "Resistor_SMD:R_0805_2012Metric_Pad1.15x1.40mm_HandSolder" V 6780 5600 50  0001 C CNN
 F 3 "https://datasheet.lcsc.com/szlcsc/1912111437_UNI-ROYAL-Uniroyal-Elec-0805W8D8201T5E_C407435.pdf" H 6850 5600 50  0001 C CNN
 F 4 "C407435" H 6850 5600 50  0001 C CNN "LCSC"
@@
 F 0 "R13" H 6920 5046 50  0000 L CNN
 F 1 "8.2kOhm" H 6920 4955 50  0000 L CNN
-F 2 "" V 6780 5000 50  0001 C CNN
+F 2 "Resistor_SMD:R_0805_2012Metric_Pad1.15x1.40mm_HandSolder" V 6780 5000 50  0001 C CNN
 F 3 "https://datasheet.lcsc.com/szlcsc/1912111437_UNI-ROYAL-Uniroyal-Elec-0805W8D8201T5E_C407435.pdf" H 6850 5000 50  0001 C CNN
 F 4 "C407435" H 6850 5000 50  0001 C CNN "LCSC"
