File: Brewnode_PCB/ADC.sch (KiCad schematic (older format))
At the start: 23 parts, among them J10 Screw_Terminal_01x03, J11 Screw_Terminal_01x03, J12 Screw_Terminal_01x03, J9 Screw_Terminal_01x03, U2 ADS1115IDGS

Commit message: More PCB Pcb work
Parts:
- C5: symbol Device:CP -> Device:C_Polarized
Changed lines of the file:
@@
 AIN3
 $Comp
-L Device:CP C5
+L Device:C_Polarized C5
 U 1 1 5F69915C
 P 7500 2850
+AR Path="/5F69915C" Ref="C5"  Part="1"
+AR Path="/5F66CC9A/5F69915C" Ref="C5"  Part="1"
 F 0 "C5" H 7618 2896 50  0000 L CNN
 F 1 "47uF" H 7618 2805 50  0000 L CNN

Commit message: Sch + PCB V1.1
Corrected FDN340 P-FET Pinout.
Added 5V, 3V3 Description in silkscreen for indication D1, D2
Parts:
- C5: symbol Device:C_Polarized -> Brewnode_PCB-rescue:C_Polarized-Device
Changed lines of the file:
@@
 Sheet 5 8
 Title "BrewnodeV1"
-Date "2020-09-16"
-Rev "1.0"
+Date "2020-10-15"
+Rev "1.1"
 Comp "Halldin"
 Comment1 "ADC"
@@
 AIN3
 $Comp
-L Device:C_Polarized C5
+L Brewnode_PCB-rescue:C_Polarized-Device C5
 U 1 1 5F69915C
 P 7500 2850
