File: Brewnode_PCB/Brewnode_PCB.sch (KiCad schematic (older format))
At the start: 0 parts

Commit message: More PCB Work
Changed lines of the file:
@@
 $Descr A4 11693 8268
 encoding utf-8
-Sheet 1 4
+Sheet 1 5
 Title "BrewnodeV1"
 Date "2020-09-14"
@@
 $EndDescr
 $Sheet
-S 7750 3350 1200 1150
+S 9000 1100 950  600
 U 5F5F1150
 F0 "IO Expander" 50
 F1 "IOExp.sch" 50
+F2 "IOExp_Int_5V" O L 9000 1550 50
+F3 "5V_IOExp_SDA" B L 9000 1400 50
+F4 "5V_IOExp_SCL" B L 9000 1250 50
+$EndSheet
+$Sheet
+S 9000 2200 950  650
+U 5F66CC9A
+F0 "ADC" 50
+F1 "ADC.sch" 50
+F2 "5V_ADC_SCL" B L 9000 2350 50
+F3 "5V_ADC_SDA" B L 9000 2500 50
+F4 "5V_ADC_RDY" B L 9000 2650 50
 $EndSheet
 $EndSCHEMATC
