File: Brewnode_PCB/Brewnode_PCB.sch (KiCad schematic (older format))
At the start: 0 parts

Commit message: More PCB Sch work
Changed lines of the file:
@@
 $Descr A4 11693 8268
 encoding utf-8
-Sheet 1 7
+Sheet 1 8
 Title "BrewnodeV1"
-Date "2020-09-15"
+Date "2020-09-16"
 Rev "1.0"
 Comp "Halldin"
@@
 $EndDescr
 $Sheet
-S 9000 1100 950  600
+S 9050 1400 950  600
 U 5F5F1150
 F0 "IO Expander" 50
 F1 "IOExp.sch" 50
-F2 "IOExp_Int_5V" O L 9000 1550 50
-F3 "5V_IOExp_SDA" B L 9000 1400 50
-F4 "5V_IOExp_SCL" B L 9000 1250 50
+F2 "IOExp_Int_5V" O L 9050 1850 50
+F3 "5V_IOExp_SDA" B L 9050 1700 50
+F4 "5V_IOExp_SCL" B L 9050 1550 50
 $EndSheet
 $Sheet
-S 9000 2200 950  650
+S 9050 2550 950  650
 U 5F66CC9A
 F0 "ADC" 50
 F1 "ADC.sch" 50
-F2 "5V_ADC_SCL" B L 9000 2350 50
-F3 "5V_ADC_SDA" B L 9000 2500 50
-F4 "5V_ADC_RDY" B L 9000 2650 50
+F2 "5V_ADC_SCL" B L 9050 2700 50
+F3 "5V_ADC_SDA" B L 9050 2850 50
+F4 "5V_ADC_RDY" B L 9050 3000 50
 $EndSheet
 $Sheet
-S 6350 1050 1100 750
+S 6400 1400 1100 750
 U 5F6162C4
 F0 "Lvl_Shifter" 50
 F1 "Lvl_Shifter.sch" 50
-F2 "LV_1" B L 6350 1200 50
-F3 "LV_2" B L 6350 1350 50
-F4 "LV_3" B L 6350 1500 50
-F5 "LV_4" B L 6350 1650 50
-F6 "HV_1" B R 7450 1200 50
-F7 "HV_2" B R 7450 1350 50
-F8 "HV_3" B R 7450 1500 50
-F9 "HV_4" B R 7450 1650 50
+F2 "LV_1" B L 6400 1550 50
+F3 "LV_2" B L 6400 1700 50
+F4 "LV_3" B L 6400 1850 50
+F5 "LV_4" B L 6400 2000 50
+F6 "HV_1" B R 7500 1550 50
+F7 "HV_2" B R 7500 1700 50
+F8 "HV_3" B R 7500 1850 50
+F9 "HV_4" B R 7500 2000 50
 $EndSheet
 $Sheet
-S 6350 2200 950  750
+S 6400 2800 950  750
 U 5F66FC6A
 F0 "Digital_Sensors" 50
 F1 "Digital_Sensors.sch" 50
-F2 "Port1" B L 6350 2350 50
-F3 "Port2" B L 6350 2500 50
-F4 "Port3" B L 6350 2650 50
-F5 "Port4" B L 6350 2800 50
+F2 "Port1" B L 6400 2950 50
+F3 "Port2" B L 6400 3100 50
+F4 "Port3" B L 6400 3250 50
+F5 "Port4" B L 6400 3400 50
 $EndSheet
+$Sheet
+S 2650 1400 1250 2250
+U 5F61AF49
+F0 "MCU_Connector" 50
+F1 "MCU_Connector.sch" 50
+F2 "5V" O R 3900 1550 100
+F3 "3V3" O R 3900 1750 100
+F4 "GND" O R 3900 1950 100
+F5 "Port1" B R 3900 2950 100
+F6 "Port2" B R 3900 3150 100
+F7 "Port3" B R 3900 3350 100
+F8 "Port4" B R 3900 3550 100
+F9 "3V3_SCL" B R 3900 2150 100
+F10 "3V3_SDA" B R 3900 2350 100
+F11 "3V3_IOExp_Int" B R 3900 2550 100
+F12 "3V3_ADC_Int" B R 3900 2750 100
+$EndSheet
+$Comp
+L power:+3V3 #PWR?
+U 1 1 5F6234F7
+P 4250 1000
+F 0 "#PWR?" H 4250 850 50  0001 C CNN
+F 1 "+3V3" H 4265 1173 50  0000 C CNN
+F 2 "" H 4250 1000 50  0001 C CNN
+F 3 "" H 4250 1000 50  0001 C CNN
+	1    4250 1000
+	1    0    0    -1
+$EndComp
+$Comp
+L power:+5V #PWR?
+U 1 1 5F6241F4
+P 4000 1000
+F 0 "#PWR?" H 4000 850 50  0001 C CNN
+F 1 "+5V" H 4015 1173 50  0000 C CNN
+F 2 "" H 4000 1000 50  0001 C CNN
+F 3 "" H 4000 1000 50  0001 C CNN
+	1    4000 1000
+	1    0    0    -1
+$EndComp
+$Comp
+L power:GND #PWR?
+U 1 1 5F6246CE
+P 4500 1300
+F 0 "#PWR?" H 4500 1050 50  0001 C CNN
+F 1 "GND" H 4505 1127 50  0000 C CNN
+F 2 "" H 4500 1300 50  0001 C CNN
+F 3 "" H 4500 1300 50  0001 C CNN
+	1    4500 1300
+	1    0    0    -1
+$EndComp
+Wire Wire Line
+	3900 1550 4000 1550
+Wire Wire Line
+	4000 1550 4000 1000
+Wire Wire Line
+	3900 1750 4250 1750
+Wire Wire Line
+	4250 1750 4250 1000
+Wire Wire Line
+	3900 1950 4350 1950
+Wire Wire Line
+	4350 1950 4350 1200
+Wire Wire Line
+	4350 1200 4500 1200
+Wire Wire Line
+	4500 1200 4500 1300
+Wire Wire Line
+	3900 2150 4900 2150
+Wire Wire Line
+	4900 2150 4900 1550
+Wire Wire Line
+	4900 1550 6400 1550
+Wire Wire Line
+	3900 2350 5000 2350
+Wire Wire Line
+	5000 2350 5000 1700
+Wire Wire Line
+	5000 1700 6400 1700
+Wire Wire Line
+	3900 2550 5100 2550
+Wire Wire Line
+	5100 2550 5100 1850
+Wire Wire Line
+	5100 1850 6400 1850
+Wire Wire Line
+	3900 2750 5200 2750
+Wire Wire Line
+	5200 2750 5200 2000
+Wire Wire Line
+	5200 2000 6400 2000
+Wire Wire Line
+	3900 3350 5800 3350
+Wire Wire Line
+	5800 3350 5800 3250
+Wire Wire Line
+	5800 3250 6400 3250
+Wire Wire Line
+	3900 3550 5900 3550
+Wire Wire Line
+	5900 3550 5900 3400
+Wire Wire Line
+	5900 3400 6400 3400
+Wire Wire Line
+	7500 2000 8000 2000
+Wire Wire Line
+	8000 2000 8000 3000
+Wire Wire Line
+	8000 3000 9050 3000
+Wire Wire Line
+	7500 1550 8600 1550
+Wire Wire Line
+	7500 1700 8450 1700
+Wire Wire Line
+	9050 1850 7500 1850
+Wire Wire Line
+	9050 2700 8600 2700
+Wire Wire Line
+	8600 2700 8600 1550
+Connection ~ 8600 1550
+Wire Wire Line
+	8600 1550 9050 1550
+Wire Wire Line
+	9050 2850 8450 2850
+Wire Wire Line
+	8450 2850 8450 1700
+Connection ~ 8450 1700
+Wire Wire Line
+	8450 1700 9050 1700
+Wire Wire Line
+	3900 3150 5700 3150
+Wire Wire Line
+	3900 2950 6400 2950
+Wire Wire Line
+	5700 3100 6400 3100
+Wire Wire Line
+	5700 3150 5700 3100
 $EndSCHEMATC

Commit message: More PCB Sch work
Parts:
- added D1, D2: LED, symbol Device:LED
- added F1, F2: Polyfuse_Small, symbol Device:Polyfuse_Small
- added R1, R2: R, symbol Device:R
Connections:
- net +3V3: now also D2.2 (A), F2.1
- net +5V: now also D1.2 (A), F1.1
- net GND: now also R1.2, R2.2
- new net: D2.1 (K), R2.1
- new net: D1.1 (K), R1.1
- new net MCU_Connector/3V3: F2.2
- new net MCU_Connector/5V: F1.2
Other:
- note added: "3V3 ON"
- note added: "5V ON"

Commit message: More PCB Sch work
Parts:
- D1, D2: value LED -> LED_1206; footprint (none) -> LED_SMD:LED_1206_3216Metric; LCSC (none) -> C125085; Mfc (none) -> LTST-C150KGKT
- F1, F2: value Polyfuse_Small -> 500mA; footprint (none) -> Fuse:Fuse_0402_1005Metric; LCSC (none) -> C206945; Mfc (none) -> 0435.500KRHF
- R1: value R -> 220Ohm; LCSC (none) -> C17557; Mfc (none) -> 0805W8F2200T5E
- R2: value R -> 100Ohm; LCSC (none) -> C17408; Mfc (none) -> 0805W8F1000T5E
Changed lines of the file:
@@
 L power:+3V3 #PWR03
 U 1 1 5F6234F7
-P 4100 900
-F 0 "#PWR03" H 4100 750 50  0001 C CNN
-F 1 "+3V3" H 4115 1073 50  0000 C CNN
-F 2 "" H 4100 900 50  0001 C CNN
-F 3 "" H 4100 900 50  0001 C CNN
-	1    4100 900
+P 5000 750
+F 0 "#PWR03" H 5000 600 50  0001 C CNN
+F 1 "+3V3" H 5015 923 50  0000 C CNN
+F 2 "" H 5000 750 50  0001 C CNN
+F 3 "" H 5000 750 50  0001 C CNN
+	1    5000 750
 	1    0    0    -1
 $EndComp
@@
 L power:+5V #PWR02
 U 1 1 5F6241F4
-P 3850 900
-F 0 "#PWR02" H 3850 750 50  0001 C CNN
-F 1 "+5V" H 3865 1073 50  0000 C CNN
-F 2 "" H 3850 900 50  0001 C CNN
-F 3 "" H 3850 900 50  0001 C CNN
-	1    3850 900
+P 4050 750
+F 0 "#PWR02" H 4050 600 50  0001 C CNN
+F 1 "+5V" H 4065 923 50  0000 C CNN
+F 2 "" H 4050 750 50  0001 C CNN
+F 3 "" H 4050 750 50  0001 C CNN
+	1    4050 750
 	1    0    0    -1
 $EndComp
@@
 P 2900 1500
 F 0 "D2" H 2893 1717 50  0000 C CNN
-F 1 "LED" H 2893 1626 50  0000 C CNN
-F 2 "" H 2900 1500 50  0001 C CNN
-F 3 "~" H 2900 1500 50  0001 C CNN
+F 1 "LED_1206" H 2893 1626 50  0000 C CNN
+F 2 "LED_SMD:LED_1206_3216Metric" H 2900 1500 50  0001 C CNN
+F 3 "https://datasheet.lcsc.com/szlcsc/1810231512_Lite-On-LTST-C150KGKT_C125085.pdf" H 2900 1500 50  0001 C CNN
+F 4 "C125085" H 2900 1500 50  0001 C CNN "LCSC"
+F 5 "LTST-C150KGKT" H 2900 1500 50  0001 C CNN "Mfc"
 	1    2900 1500
 	1    0    0    -1
@@
 P 2900 1100
 F 0 "D1" H 2893 1317 50  0000 C CNN
-F 1 "LED" H 2893 1226 50  0000 C CNN
-F 2 "" H 2900 1100 50  0001 C CNN
-F 3 "~" H 2900 1100 50  0001 C CNN
+F 1 "LED_1206" H 2893 1226 50  0000 C CNN
+F 2 "LED_SMD:LED_1206_3216Metric" H 2900 1100 50  0001 C CNN
+F 3 "https://datasheet.lcsc.com/szlcsc/1810231512_Lite-On-LTST-C150KGKT_C125085.pdf" H 2900 1100 50  0001 C CNN
+F 4 "C125085" H 2900 1100 50  0001 C CNN "LCSC"
+F 5 "LTST-C150KGKT" H 2900 1100 50  0001 C CNN "Mfc"
 	1    2900 1100
 	1    0    0    -1
@@
 P 3850 1300
 F 0 "F1" H 3700 1400 50  0000 L CNN
-F 1 "Polyfuse_Small" H 3250 1300 50  0000 L CNN
-F 2 "" H 3900 1100 50  0001 L CNN
-F 3 "~" H 3850 1300 50  0001 C CNN
+F 1 "500mA" H 3500 1300 50  0000 L CNN
+F 2 "Fuse:Fuse_0402_1005Metric" H 3900 1100 50  0001 L CNN
+F 3 "https://datasheet.lcsc.com/szlcsc/1808141123_Littelfuse-0435-500KRHF_C206945.pdf" H 3850 1300 50  0001 C CNN
+F 4 "C206945" H 3850 1300 50  0001 C CNN "LCSC"
+F 5 "0435.500KRHF" H 3850 1300 50  0001 C CNN "Mfc"
 	1    3850 1300
 	1    0    0    -1
@@
 P 4100 1650
 F 0 "F2" H 4168 1696 50  0000 L CNN
-F 1 "Polyfuse_Small" H 4168 1605 50  0000 L CNN
-F 2 "" H 4150 1450 50  0001 L CNN
-F 3 "~" H 4100 1650 50  0001 C CNN
+F 1 "500mA" H 4168 1605 50  0000 L CNN
+F 2 "Fuse:Fuse_0402_1005Metric" H 4150 1450 50  0001 L CNN
+F 3 "https://datasheet.lcsc.com/szlcsc/1808141123_Littelfuse-0435-500KRHF_C206945.pdf" H 4100 1650 50  0001 C CNN
+F 4 "C206945" H 4100 1650 50  0001 C CNN "LCSC"
+F 5 "0435.500KRHF" H 4100 1650 50  0001 C CNN "Mfc"
 	1    4100 1650
 	1    0    0    -1
@@
 P 2400 1100
 F 0 "R1" V 2193 1100 50  0000 C CNN
-F 1 "R" V 2284 1100 50  0000 C CNN
+F 1 "220Ohm" V 2284 1100 50  0000 C CNN
 F 2 "" V 2330 1100 50  0001 C CNN
-F 3 "~" H 2400 1100 50  0001 C CNN
+F 3 "https://datasheet.lcsc.com/szlcsc/1810241809_UNI-ROYAL-Uniroyal-Elec-0805W8F2200T5E_C17557.pdf" H 2400 1100 50  0001 C CNN
+F 4 "C17557" H 2400 1100 50  0001 C CNN "LCSC"
+F 5 "0805W8F2200T5E" H 2400 1100 50  0001 C CNN "Mfc"
 	1    2400 1100
 	0    1    1    0
@@
 $EndComp
 Wire Wire Line
-	4100 1750 4100 2600
-Wire Wire Line
 	4100 1550 4100 1500
 Wire Wire Line
-	3850 900  3850 1100
-Wire Wire Line
-	3850 1400 3850 2400
+	4050 750  4050 950
 $Comp
 L Device:R R2
@@
 P 2400 1500
 F 0 "R2" V 2193 1500 50  0000 C CNN
-F 1 "R" V 2284 1500 50  0000 C CNN
+F 1 "100Ohm" V 2284 1500 50  0000 C CNN
 F 2 "" V 2330 1500 50  0001 C CNN
-F 3 "~" H 2400 1500 50  0001 C CNN
+F 3 "https://datasheet.lcsc.com/szlcsc/1809062111_UNI-ROYAL-Uniroyal-Elec-0805W8F1000T5E_C17408.pdf" H 2400 1500 50  0001 C CNN
+F 4 "C17408" H 2400 1500 50  0001 C CNN "LCSC"
+F 5 "0805W8F1000T5E" H 2400 1500 50  0001 C CNN "Mfc"
 	1    2400 1500
 	0    1    1    0
@@
 Wire Wire Line
 	3050 1100 3850 1100
-Connection ~ 3850 1100
 Wire Wire Line
 	3850 1100 3850 1200
 Wire Wire Line
 	3050 1500 4100 1500
-Connection ~ 4100 1500
-Wire Wire Line
-	4100 1500 4100 900
+Wire Wire Line
+	5000 1350 5000 850
 Text Notes 2800 850  0    50   ~ 0
 5V ON
 Text Notes 2800 1700 0    50   ~ 0
 3V3 ON
+Wire Wire Line
+	4100 1750 4100 2600
+Wire Wire Line
+	3850 1400 3850 2400
+$Comp
+L power:PWR_FLAG #FLG0101
+U 1 1 5F651973
+P 4300 850
+F 0 "#FLG0101" H 4300 925 50  0001 C CNN
+F 1 "PWR_FLAG" H 4300 1023 50  0000 C CNN
+F 2 "" H 4300 850 50  0001 C CNN
+F 3 "~" H 4300 850 50  0001 C CNN
+	1    4300 850
+	1    0    0    -1
+$EndComp
+$Comp
+L power:PWR_FLAG #FLG0102
+U 1 1 5F6521CD
+P 5250 850
+F 0 "#FLG0102" H 5250 925 50  0001 C CNN
+F 1 "PWR_FLAG" H 5250 1023 50  0000 C CNN
+F 2 "" H 5250 850 50  0001 C CNN
+F 3 "~" H 5250 850 50  0001 C CNN
+	1    5250 850
+	1    0    0    -1
+$EndComp
+$Comp
+L power:PWR_FLAG #FLG0103
+U 1 1 5F653407
+P 4700 2050
+F 0 "#FLG0103" H 4700 2125 50  0001 C CNN
+F 1 "PWR_FLAG" H 4700 2223 50  0000 C CNN
+F 2 "" H 4700 2050 50  0001 C CNN
+F 3 "~" H 4700 2050 50  0001 C CNN
+	1    4700 2050
+	1    0    0    -1
+$EndComp
+Wire Wire Line
+	5000 1350 4100 1350
+Wire Wire Line
+	4100 1350 4100 1500
+Connection ~ 4100 1500
+Wire Wire Line
+	5250 850  5000 850
+Connection ~ 5000 850
+Wire Wire Line
+	5000 850  5000 750
+Wire Wire Line
+	4050 950  3850 950
+Wire Wire Line
+	3850 950  3850 1100
+Connection ~ 3850 1100
+Wire Wire Line
+	4300 850  4300 950
+Wire Wire Line
+	4300 950  4050 950
+Connection ~ 4050 950
+Wire Wire Line
+	4700 2050 4350 2050
+Connection ~ 4350 2050
 $EndSCHEMATC

Commit message: Done PCB Sch Work
Parts:
- R1, R2: footprint (none) -> Resistor_SMD:R_0805_2012Metric_Pad1.15x1.40mm_HandSolder
Changed lines of the file:
@@
 F 0 "R1" V 2193 1100 50  0000 C CNN
 F 1 "220Ohm" V 2284 1100 50  0000 C CNN
-F 2 "" V 2330 1100 50  0001 C CNN
+F 2 "Resistor_SMD:R_0805_2012Metric_Pad1.15x1.40mm_HandSolder" V 2330 1100 50  0001 C CNN
 F 3 "https://datasheet.lcsc.com/szlcsc/1810241809_UNI-ROYAL-Uniroyal-Elec-0805W8F2200T5E_C17557.pdf" H 2400 1100 50  0001 C CNN
 F 4 "C17557" H 2400 1100 50  0001 C CNN "LCSC"
@@
 F 0 "R2" V 2193 1500 50  0000 C CNN
 F 1 "100Ohm" V 2284 1500 50  0000 C CNN
-F 2 "" V 2330 1500 50  0001 C CNN
+F 2 "Resistor_SMD:R_0805_2012Metric_Pad1.15x1.40mm_HandSolder" V 2330 1500 50  0001 C CNN
 F 3 "https://datasheet.lcsc.com/szlcsc/1809062111_UNI-ROYAL-Uniroyal-Elec-0805W8F1000T5E_C17408.pdf" H 2400 1500 50  0001 C CNN
 F 4 "C17408" H 2400 1500 50  0001 C CNN "LCSC"

Commit message: More PCB Pcb work
Other:
- moved on the sheet: D1, D2, F1, F2, R1, R2
