File: Brewnode_PCB/IOExp.sch (KiCad schematic (older format))
At the start: 1 part

Commit message: More PCB Work
Parts:
- added C?: C, symbol Device:C
Connections:
- net IOExp_P0 is gone; now on net IOExp_Inputs/Input_1: U?.4 (P0)
- net IOExp_P1 is gone; now on net IOExp_Inputs/Input_2: U?.5 (P1)
- net IOExp_P2 is gone; now on net IOExp_Inputs/Input_3: U?.6 (P2)
- net IOExp_P3 is gone; now on net IOExp_Inputs/Input_4: U?.7 (P3)
- net +5V: now also C?.1
- net GND: now also C?.2
- net 5V_SCL renamed 5V_IOExp_SCL
- net 5V_SDA renamed 5V_IOExp_SDA
- net IOExp_P4 renamed IOExp_Relays/Output_1
- net IOExp_P5 renamed IOExp_Relays/Output_2
- net IOExp_P6 renamed IOExp_Relays/Output_3
- net IOExp_P7 renamed IOExp_Relays/Output_4
Changed lines of the file:
@@
 $Descr A4 11693 8268
 encoding utf-8
-Sheet 2 4
+Sheet 2 5
 Title "BrewnodeV1"
 Date "2020-09-14"
@@
 $EndComp
 Text HLabel 3650 3900 0    50   BiDi ~ 0
-5V_SDA
+5V_IOExp_SDA
 Text HLabel 3650 3700 0    50   BiDi ~ 0
-5V_SCL
+5V_IOExp_SCL
 $Comp
 L power:+5V #PWR0101
@@
 	4000 3850 4400 3850
 Wire Wire Line
-	4900 3450 4900 3000
+	4900 3450 4900 3100
 Wire Wire Line
 	4900 4850 4900 5050
@@
 Wire Wire Line
 	4150 4250 4150 5050
-Text HLabel 6400 3750 2    50   Input ~ 0
-IOExp_P0
-Text HLabel 6400 3850 2    50   Input ~ 0
-IOExp_P1
-Text HLabel 6400 3950 2    50   Input ~ 0
-IOExp_P2
-Text HLabel 6400 4050 2    50   Input ~ 0
-IOExp_P3
-Text HLabel 6000 4150 2    50   Output ~ 0
-IOExp_P4
-Text HLabel 6000 4250 2    50   Output ~ 0
-IOExp_P5
-Text HLabel 6000 4350 2    50   Output ~ 0
-IOExp_P6
-Text HLabel 6000 4450 2    50   Output ~ 0
-IOExp_P7
-Wire Wire Line
-	5400 3750 6400 3750
-Wire Wire Line
-	5400 3950 6400 3950
-Wire Wire Line
-	5400 4150 6000 4150
-Wire Wire Line
-	5400 4250 6000 4250
-Wire Wire Line
-	5400 4350 6000 4350
-Wire Wire Line
-	5400 4450 6000 4450
-Wire Wire Line
-	5400 3850 6400 3850
-Wire Wire Line
-	5400 4050 6400 4050
 Text HLabel 3650 4550 0    50   Output ~ 0
 IOExp_Int_5V
@@
 	3650 4550 4400 4550
 $Sheet
-S 7850 3150 1150 750
+S 7850 3200 850  500
 U 5F5FA99D
 F0 "IOExp_Inputs" 50
 F1 "IOExp_Inputs.sch" 50
 F2 "Input_1" B L 7850 3300 50
-F3 "Input_2" B L 7850 3450 50
-F4 "Input_3" B L 7850 3600 50
-F5 "Input_4" B L 7850 3750 50
+F3 "Input_2" B L 7850 3400 50
+F4 "Input_3" B L 7850 3500 50
+F5 "Input_4" B L 7850 3600 50
 $EndSheet
 $Sheet
-S 7850 4350 1150 850
+S 7850 4300 850  500
 U 5F5FAAA5
 F0 "IOExp_Relays" 50
 F1 "IOExp_Relays.sch" 50
+F2 "Output_1" B L 7850 4400 50
+F3 "Output_2" B L 7850 4500 50
+F4 "Output_3" B L 7850 4600 50
+F5 "Output_4" B L 7850 4700 50
 $EndSheet
+Wire Wire Line
+	5400 3750 6450 3750
+Wire Wire Line
+	6450 3750 6450 3300
+Wire Wire Line
+	6450 3300 7850 3300
+Wire Wire Line
+	5400 3850 6550 3850
+Wire Wire Line
+	6550 3850 6550 3400
+Wire Wire Line
+	6550 3400 7850 3400
+Wire Wire Line
+	5400 3950 6650 3950
+Wire Wire Line
+	6650 3950 6650 3500
+Wire Wire Line
+	6650 3500 7850 3500
+Wire Wire Line
+	5400 4050 6750 4050
+Wire Wire Line
+	6750 4050 6750 3600
+Wire Wire Line
+	6750 3600 7850 3600
+Wire Wire Line
+	5400 4150 6750 4150
+Wire Wire Line
+	6750 4150 6750 4400
+Wire Wire Line
+	6750 4400 7850 4400
+Wire Wire Line
+	5400 4250 6650 4250
+Wire Wire Line
+	6650 4250 6650 4500
+Wire Wire Line
+	6650 4500 7850 4500
+Wire Wire Line
+	5400 4350 6550 4350
+Wire Wire Line
+	6550 4350 6550 4600
+Wire Wire Line
+	6550 4600 7850 4600
+Wire Wire Line
+	5400 4450 6450 4450
+Wire Wire Line
+	6450 4450 6450 4700
+Wire Wire Line
+	6450 4700 7850 4700
+$Comp
+L Device:C C?
+U 1 1 5F66D058
+P 2800 4050
+F 0 "C?" H 2915 4096 50  0000 L CNN
+F 1 "C" H 2915 4005 50  0000 L CNN
+F 2 "" H 2838 3900 50  0001 C CNN
+F 3 "~" H 2800 4050 50  0001 C CNN
+	1    2800 4050
+	1    0    0    -1
+$EndComp
+Wire Wire Line
+	2800 3900 2800 3100
+Wire Wire Line
+	2800 3100 4900 3100
+Connection ~ 4900 3100
+Wire Wire Line
+	4900 3100 4900 3000
+Wire Wire Line
+	2800 4200 2800 5050
+Wire Wire Line
+	2800 5050 4150 5050
+Connection ~ 4150 5050
 $EndSCHEMATC
