File: Brewnode_PCB/IOExp.sch (KiCad schematic (older format))
At the start: 2 parts

Commit message: More PCB Sch work
Parts:
- gave numbers to parts that had none: 2
Changed lines of the file:
@@
 $EndDescr
 $Comp
-L Interface_Expansion:PCF8574 U?
+L Interface_Expansion:PCF8574 U1
 U 1 1 5F5F2794
 P 4900 4150
-F 0 "U?" H 4900 5031 50  0000 C CNN
-F 1 "PCF8574" H 4900 4940 50  0000 C CNN
+F 0 "U1" H 5000 5000 50  0000 C CNN
+F 1 "PCF8574" H 5100 4900 50  0000 C CNN
 F 2 "" H 4900 4150 50  0001 C CNN
 F 3 "http://www.nxp.com/documents/data_sheet/PCF8574_PCF8574A.pdf" H 4900 4150 50  0001 C CNN
@@
 5V_IOExp_SCL
 $Comp
-L power:+5V #PWR0101
+L power:+5V #PWR05
 U 1 1 5F5F3853
 P 4900 3000
-F 0 "#PWR0101" H 4900 2850 50  0001 C CNN
+F 0 "#PWR05" H 4900 2850 50  0001 C CNN
 F 1 "+5V" H 4915 3173 50  0000 C CNN
 F 2 "" H 4900 3000 50  0001 C CNN
@@
 $EndComp
 $Comp
-L power:GND #PWR0102
+L power:GND #PWR06
 U 1 1 5F5F3EF2
 P 4900 5150
-F 0 "#PWR0102" H 4900 4900 50  0001 C CNN
+F 0 "#PWR06" H 4900 4900 50  0001 C CNN
 F 1 "GND" H 4905 4977 50  0000 C CNN
 F 2 "" H 4900 5150 50  0001 C CNN
@@
 	6450 4700 7850 4700
 $Comp
-L Device:C C?
+L Device:C C1
 U 1 1 5F66D058
 P 2800 4050
-F 0 "C?" H 2915 4096 50  0000 L CNN
+F 0 "C1" H 2915 4096 50  0000 L CNN
 F 1 "C" H 2915 4005 50  0000 L CNN
 F 2 "" H 2838 3900 50  0001 C CNN

Commit message: More PCB Sch work
Parts:
- C1: value C -> 100nF; footprint (none) -> Capacitor_SMD:C_0402_1005Metric; LCSC (none) -> C1525; Mfc (none) -> CL05B104KO5NNNC
- U1: LCSC (none) -> C7605; Mfc (none) -> PCF8574T/3,518
Changed lines of the file:
@@
 F 1 "PCF8574" H 5100 4900 50  0000 C CNN
 F 2 "" H 4900 4150 50  0001 C CNN
-F 3 "http://www.nxp.com/documents/data_sheet/PCF8574_PCF8574A.pdf" H 4900 4150 50  0001 C CNN
+F 3 "https://datasheet.lcsc.com/szlcsc/1809261711_NXP-Semicon-PCF8574T-3-518_C7605.pdf" H 4900 4150 50  0001 C CNN
+F 4 "C7605" H 4900 4150 50  0001 C CNN "LCSC"
+F 5 "PCF8574T/3,518" H 4900 4150 50  0001 C CNN "Mfc"
 	1    4900 4150
 	1    0    0    -1
@@
 P 2800 4050
 F 0 "C1" H 2915 4096 50  0000 L CNN
-F 1 "C" H 2915 4005 50  0000 L CNN
-F 2 "" H 2838 3900 50  0001 C CNN
-F 3 "~" H 2800 4050 50  0001 C CNN
+F 1 "100nF" H 2915 4005 50  0000 L CNN
+F 2 "Capacitor_SMD:C_0402_1005Metric" H 2838 3900 50  0001 C CNN
+F 3 "https://datasheet.lcsc.com/szlcsc/1810191219_Samsung-Electro-Mechanics-CL05B104KO5NNNC_C1525.pdf" H 2800 4050 50  0001 C CNN
+F 4 "C1525" H 2800 4050 50  0001 C CNN "LCSC"
+F 5 "CL05B104KO5NNNC" H 2800 4050 50  0001 C CNN "Mfc"
 	1    2800 4050
 	1    0    0    -1

Commit message: Done PCB Sch Work
Parts:
- U1: footprint (none) -> Package_SO:SOIC-16W_7.5x10.3mm_P1.27mm
Changed lines of the file:
@@
 F 0 "U1" H 5000 5000 50  0000 C CNN
 F 1 "PCF8574" H 5100 4900 50  0000 C CNN
-F 2 "" H 4900 4150 50  0001 C CNN
+F 2 "Package_SO:SOIC-16W_7.5x10.3mm_P1.27mm" H 4900 4150 50  0001 C CNN
 F 3 "https://datasheet.lcsc.com/szlcsc/1809261711_NXP-Semicon-PCF8574T-3-518_C7605.pdf" H 4900 4150 50  0001 C CNN
 F 4 "C7605" H 4900 4150 50  0001 C CNN "LCSC"

Commit message: PCB  V1 To production
Changed lines of the file:
@@
 Text HLabel 3650 4550 0    50   Output ~ 0
 IOExp_Int_5V
-Wire Wire Line
-	3650 4550 4400 4550
 $Sheet
 S 7850 3200 850  500
@@
 	2800 5050 4150 5050
 Connection ~ 4150 5050
+Wire Wire Line
+	4400 4550 3650 4550
 $EndSCHEMATC
