File: Brewnode_PCB/IOExp_Inputs.sch (KiCad schematic (older format))
At the start: 4 parts

Commit message: More PCB Work
Parts:
- added C?: CP, symbol Device:CP
Connections:
- net +5V: now also C?.1
- net GND: now also C?.2
Changed lines of the file:
@@
 $Descr A4 11693 8268
 encoding utf-8
-Sheet 3 4
+Sheet 3 5
 Title ""
 Date ""
@@
 Wire Wire Line
 	6850 4100 8000 4100
+$Comp
+L Device:CP C?
+U 1 1 5F69BB32
+P 5800 3350
+F 0 "C?" H 5918 3396 50  0000 L CNN
+F 1 "CP" H 5918 3305 50  0000 L CNN
+F 2 "" H 5838 3200 50  0001 C CNN
+F 3 "~" H 5800 3350 50  0001 C CNN
+	1    5800 3350
+	1    0    0    -1
+$EndComp
+Wire Wire Line
+	5800 3200 5800 2500
+Wire Wire Line
+	5800 2500 7650 2500
+Wire Wire Line
+	5800 3500 5800 4200
+Wire Wire Line
+	5800 4200 7500 4200
 $EndSCHEMATC
