File: Brewnode_PCB/IOExp_Relays.sch (KiCad schematic (older format))
At the start: 17 parts

Commit message: More PCB Work
Parts:
- removed D? (x3): D, symbol Device:D
- removed J? (x3): Screw_Terminal_01x03, symbol Connector:Screw_Terminal_01x03
- removed K? (x3): SANYOU_SRD_Form_C, Relay_THT:Relay_SPDT_SANYOU_SRD_Series_Form_C, symbol Relay:SANYOU_SRD_Form_C
- removed Q? (x4): IRLIZ44N, Package_TO_SOT_THT:TO-220F-3_Vertical, symbol Transistor_FET:IRLIZ44N
- removed R?: R, symbol Device:R
- added C?: CP, symbol Device:CP
- added D? (x3): D, symbol Device:D
- added J? (x3): Screw_Terminal_01x03, symbol Connector:Screw_Terminal_01x03
- added K? (x3): SANYOU_SRD_Form_C, Relay_THT:Relay_SPDT_SANYOU_SRD_Series_Form_C, symbol Relay:SANYOU_SRD_Form_C
- added Q? (x4): FDN340P, Package_TO_SOT_SMD:SOT-23, symbol Transistor_FET:FDN340P
- added R? (x4): R, symbol Device:R
Connections:
- net labels added: Output_2, Output_3, Output_4
- wire segments 76 -> 118
Other:
- moved on the sheet: D?, J?, K?
