File: Brewnode_PCB/IOExp_Relays.sch (KiCad schematic (older format))
At the start: 21 parts

Commit message: More PCB Sch work
Parts:
- gave numbers to parts that had none: 21
Changed lines of the file:
@@
 $EndDescr
 $Comp
-L Relay:SANYOU_SRD_Form_C K?
+L Relay:SANYOU_SRD_Form_C K1
 U 1 1 5F643939
 P 3150 2450
-F 0 "K?" H 3580 2496 50  0000 L CNN
+F 0 "K1" H 3580 2496 50  0000 L CNN
 F 1 "SANYOU_SRD_Form_C" H 3580 2405 50  0000 L CNN
 F 2 "Relay_THT:Relay_SPDT_SANYOU_SRD_Series_Form_C" H 3600 2400 50  0001 L CNN
@@
 $EndComp
 $Comp
-L power:+5V #PWR?
+L power:+5V #PWR09
 U 1 1 5F64C92B
 P 2950 1400
-F 0 "#PWR?" H 2950 1250 50  0001 C CNN
+F 0 "#PWR09" H 2950 1250 50  0001 C CNN
 F 1 "+5V" H 2965 1573 50  0000 C CNN
 F 2 "" H 2950 1400 50  0001 C CNN
@@
 $EndComp
 $Comp
-L Device:D D?
+L Device:D D3
 U 1 1 5F64D292
 P 2350 2450
-F 0 "D?" V 2304 2530 50  0000 L CNN
+F 0 "D3" V 2304 2530 50  0000 L CNN
 F 1 "D" V 2395 2530 50  0000 L CNN
 F 2 "" H 2350 2450 50  0001 C CNN
@@
 $EndComp
 $Comp
-L power:GND #PWR?
+L power:GND #PWR010
 U 1 1 5F64EBA7
 P 2950 3000
-F 0 "#PWR?" H 2950 2750 50  0001 C CNN
+F 0 "#PWR010" H 2950 2750 50  0001 C CNN
 F 1 "GND" H 2955 2827 50  0000 C CNN
 F 2 "" H 2950 3000 50  0001 C CNN
@@
 Output_1
 $Comp
-L Transistor_FET:FDN340P Q?
+L Transistor_FET:FDN340P Q1
 U 1 1 5F60DD24
 P 2850 1850
-F 0 "Q?" H 3054 1896 50  0000 L CNN
+F 0 "Q1" H 3054 1896 50  0000 L CNN
 F 1 "FDN340P" H 3054 1805 50  0000 L CNN
 F 2 "Package_TO_SOT_SMD:SOT-23" H 3050 1775 50  0001 L CIN
@@
 $EndComp
 $Comp
-L Device:R R?
+L Device:R R3
 U 1 1 5F610E39
 P 2500 1500
-F 0 "R?" H 2570 1546 50  0000 L CNN
+F 0 "R3" H 2570 1546 50  0000 L CNN
 F 1 "R" H 2570 1455 50  0000 L CNN
 F 2 "" V 2430 1500 50  0001 C CNN
@@
 	3250 2000 3450 2000
 $Comp
-L Connector:Screw_Terminal_01x03 J?
+L Connector:Screw_Terminal_01x03 J5
 U 1 1 5F64B72A
 P 4050 1950
-F 0 "J?" H 4130 1992 50  0000 L CNN
+F 0 "J5" H 4130 1992 50  0000 L CNN
 F 1 "Screw_Terminal_01x03" H 4130 1901 50  0000 L CNN
 F 2 "" H 4050 1950 50  0001 C CNN
@@
 Connection ~ 2500 1850
 $Comp
-L Relay:SANYOU_SRD_Form_C K?
+L Relay:SANYOU_SRD_Form_C K3
 U 1 1 5F62CCBA
 P 8050 2450
-F 0 "K?" H 8480 2496 50  0000 L CNN
+F 0 "K3" H 8480 2496 50  0000 L CNN
 F 1 "SANYOU_SRD_Form_C" H 8480 2405 50  0000 L CNN
 F 2 "Relay_THT:Relay_SPDT_SANYOU_SRD_Series_Form_C" H 8500 2400 50  0001 L CNN
@@
 $EndComp
 $Comp
-L power:+5V #PWR?
+L power:+5V #PWR015
 U 1 1 5F62CCC0
 P 7850 1400
-F 0 "#PWR?" H 7850 1250 50  0001 C CNN
+F 0 "#PWR015" H 7850 1250 50  0001 C CNN
 F 1 "+5V" H 7865 1573 50  0000 C CNN
 F 2 "" H 7850 1400 50  0001 C CNN
@@
 $EndComp
 $Comp
-L Device:D D?
+L Device:D D5
 U 1 1 5F62CCC6
 P 7250 2450
-F 0 "D?" V 7204 2530 50  0000 L CNN
+F 0 "D5" V 7204 2530 50  0000 L CNN
 F 1 "D" V 7295 2530 50  0000 L CNN
 F 2 "" H 7250 2450 50  0001 C CNN
@@
 $EndComp
 $Comp
-L power:GND #PWR?
+L power:GND #PWR016
 U 1 1 5F62CCCC
 P 7850 3000
-F 0 "#PWR?" H 7850 2750 50  0001 C CNN
+F 0 "#PWR016" H 7850 2750 50  0001 C CNN
 F 1 "GND" H 7855 2827 50  0000 C CNN
 F 2 "" H 7850 3000 50  0001 C CNN
@@
 Output_2
 $Comp
-L Transistor_FET:FDN340P Q?
+L Transistor_FET:FDN340P Q3
 U 1 1 5F62CCD3
 P 7750 1850
-F 0 "Q?" H 7954 1896 50  0000 L CNN
+F 0 "Q3" H 7954 1896 50  0000 L CNN
 F 1 "FDN340P" H 7954 1805 50  0000 L CNN
 F 2 "Package_TO_SOT_SMD:SOT-23" H 7950 1775 50  0001 L CIN
@@
 $EndComp
 $Comp
-L Device:R R?
+L Device:R R5
 U 1 1 5F62CCD9
 P 7400 1500
-F 0 "R?" H 7470 1546 50  0000 L CNN
+F 0 "R5" H 7470 1546 50  0000 L CNN
 F 1 "R" H 7470 1455 50  0000 L CNN
 F 2 "" V 7330 1500 50  0001 C CNN
@@
 	8150 2000 8350 2000
 $Comp
-L Connector:Screw_Terminal_01x03 J?
+L Connector:Screw_Terminal_01x03 J7
 U 1 1 5F62CCE7
 P 8950 1950
-F 0 "J?" H 9030 1992 50  0000 L CNN
+F 0 "J7" H 9030 1992 50  0000 L CNN
 F 1 "Screw_Terminal_01x03" H 9030 1901 50  0000 L CNN
 F 2 "" H 8950 1950 50  0001 C CNN
@@
 Connection ~ 7400 1850
 $Comp
-L Relay:SANYOU_SRD_Form_C K?
+L Relay:SANYOU_SRD_Form_C K2
 U 1 1 5F634AB0
 P 3150 5100
-F 0 "K?" H 3580 5146 50  0000 L CNN
+F 0 "K2" H 3580 5146 50  0000 L CNN
 F 1 "SANYOU_SRD_Form_C" H 3580 5055 50  0000 L CNN
 F 2 "Relay_THT:Relay_SPDT_SANYOU_SRD_Series_Form_C" H 3600 5050 50  0001 L CNN
@@
 $EndComp
 $Comp
-L power:+5V #PWR?
+L power:+5V #PWR011
 U 1 1 5F634AB6
 P 2950 4050
-F 0 "#PWR?" H 2950 3900 50  0001 C CNN
+F 0 "#PWR011" H 2950 3900 50  0001 C CNN
 F 1 "+5V" H 2965 4223 50  0000 C CNN
 F 2 "" H 2950 4050 50  0001 C CNN
@@
 $EndComp
 $Comp
-L Device:D D?
+L Device:D D4
 U 1 1 5F634ABC
 P 2350 5100
-F 0 "D?" V 2304 5180 50  0000 L CNN
+F 0 "D4" V 2304 5180 50  0000 L CNN
 F 1 "D" V 2395 5180 50  0000 L CNN
 F 2 "" H 2350 5100 50  0001 C CNN
@@
 $EndComp
 $Comp
-L power:GND #PWR?
+L power:GND #PWR012
 U 1 1 5F634AC2
 P 2950 5650
-F 0 "#PWR?" H 2950 5400 50  0001 C CNN
+F 0 "#PWR012" H 2950 5400 50  0001 C CNN
 F 1 "GND" H 2955 5477 50  0000 C CNN
 F 2 "" H 2950 5650 50  0001 C CNN
@@
 Output_3
 $Comp
-L Transistor_FET:FDN340P Q?
+L Transistor_FET:FDN340P Q2
 U 1 1 5F634AC9
 P 2850 4500
-F 0 "Q?" H 3054 4546 50  0000 L CNN
+F 0 "Q2" H 3054 4546 50  0000 L CNN
 F 1 "FDN340P" H 3054 4455 50  0000 L CNN
 F 2 "Package_TO_SOT_SMD:SOT-23" H 3050 4425 50  0001 L CIN
@@
 $EndComp
 $Comp
-L Device:R R?
+L Device:R R4
 U 1 1 5F634ACF
 P 2500 4150
-F 0 "R?" H 2570 4196 50  0000 L CNN
+F 0 "R4" H 2570 4196 50  0000 L CNN
 F 1 "R" H 2570 4105 50  0000 L CNN
 F 2 "" V 2430 4150 50  0001 C CNN
@@
 	3250 4650 3450 4650
 $Comp
-L Connector:Screw_Terminal_01x03 J?
+L Connector:Screw_Terminal_01x03 J6
 U 1 1 5F634ADD
 P 4050 4600
-F 0 "J?" H 4130 4642 50  0000 L CNN
+F 0 "J6" H 4130 4642 50  0000 L CNN
 F 1 "Screw_Terminal_01x03" H 4130 4551 50  0000 L CNN
 F 2 "" H 4050 4600 50  0001 C CNN
@@
 Connection ~ 2500 4500
 $Comp
-L Relay:SANYOU_SRD_Form_C K?
+L Relay:SANYOU_SRD_Form_C K4
 U 1 1 5F6409D1
 P 8050 5100
-F 0 "K?" H 8480 5146 50  0000 L CNN
+F 0 "K4" H 8480 5146 50  0000 L CNN
 F 1 "SANYOU_SRD_Form_C" H 8480 5055 50  0000 L CNN
 F 2 "Relay_THT:Relay_SPDT_SANYOU_SRD_Series_Form_C" H 8500 5050 50  0001 L CNN
@@
 $EndComp
 $Comp
-L power:+5V #PWR?
+L power:+5V #PWR017
 U 1 1 5F6409D7
 P 7850 4050
-F 0 "#PWR?" H 7850 3900 50  0001 C CNN
+F 0 "#PWR017" H 7850 3900 50  0001 C CNN
 F 1 "+5V" H 7865 4223 50  0000 C CNN
 F 2 "" H 7850 4050 50  0001 C CNN
@@
 $EndComp
 $Comp
-L Device:D D?
+L Device:D D6
 U 1 1 5F6409DD
 P 7250 5100
-F 0 "D?" V 7204 5180 50  0000 L CNN
+F 0 "D6" V 7204 5180 50  0000 L CNN
 F 1 "D" V 7295 5180 50  0000 L CNN
 F 2 "" H 7250 5100 50  0001 C CNN
@@
 $EndComp
 $Comp
-L power:GND #PWR?
+L power:GND #PWR018
 U 1 1 5F6409E3
 P 7850 5650
-F 0 "#PWR?" H 7850 5400 50  0001 C CNN
+F 0 "#PWR018" H 7850 5400 50  0001 C CNN
 F 1 "GND" H 7855 5477 50  0000 C CNN
 F 2 "" H 7850 5650 50  0001 C CNN
@@
 Output_4
 $Comp
-L Transistor_FET:FDN340P Q?
+L Transistor_FET:FDN340P Q4
 U 1 1 5F6409EA
 P 7750 4500
-F 0 "Q?" H 7954 4546 50  0000 L CNN
+F 0 "Q4" H 7954 4546 50  0000 L CNN
 F 1 "FDN340P" H 7954 4455 50  0000 L CNN
 F 2 "Package_TO_SOT_SMD:SOT-23" H 7950 4425 50  0001 L CIN
@@
 $EndComp
 $Comp
-L Device:R R?
+L Device:R R6
 U 1 1 5F6409F0
 P 7400 4150
-F 0 "R?" H 7470 4196 50  0000 L CNN
+F 0 "R6" H 7470 4196 50  0000 L CNN
 F 1 "R" H 7470 4105 50  0000 L CNN
 F 2 "" V 7330 4150 50  0001 C CNN
@@
 	8150 4650 8350 4650
 $Comp
-L Connector:Screw_Terminal_01x03 J?
+L Connector:Screw_Terminal_01x03 J8
 U 1 1 5F6409FE
 P 8950 4600
-F 0 "J?" H 9030 4642 50  0000 L CNN
+F 0 "J8" H 9030 4642 50  0000 L CNN
 F 1 "Screw_Terminal_01x03" H 9030 4551 50  0000 L CNN
 F 2 "" H 8950 4600 50  0001 C CNN
@@
 Connection ~ 7400 4500
 $Comp
-L Device:CP C?
+L Device:CP C3
 U 1 1 5F69DC17
 P 5850 3400
-F 0 "C?" H 5968 3446 50  0000 L CNN
+F 0 "C3" H 5968 3446 50  0000 L CNN
 F 1 "CP" H 5968 3355 50  0000 L CNN
 F 2 "" H 5888 3250 50  0001 C CNN
@@
 $EndComp
 $Comp
-L power:+5V #PWR?
+L power:+5V #PWR013
 U 1 1 5F69EA52
 P 5850 3100
-F 0 "#PWR?" H 5850 2950 50  0001 C CNN
+F 0 "#PWR013" H 5850 2950 50  0001 C CNN
 F 1 "+5V" H 5865 3273 50  0000 C CNN
 F 2 "" H 5850 3100 50  0001 C CNN
@@
 $EndComp
 $Comp
-L power:GND #PWR?
+L power:GND #PWR014
 U 1 1 5F69F3F2
 P 5850 3700
-F 0 "#PWR?" H 5850 3450 50  0001 C CNN
+F 0 "#PWR014" H 5850 3450 50  0001 C CNN
 F 1 "GND" H 5855 3527 50  0000 C CNN
 F 2 "" H 5850 3700 50  0001 C CNN

Commit message: More PCB Sch work
Parts:
- C3: value CP -> 220uF; footprint (none) -> Capacitor_SMD:CP_Elec_8x10; LCSC (none) -> C249801; Mfc (none) -> VUA221M1ATR-0810
- D3, D4, D5, D6: value D -> SMA; footprint (none) -> Diode_SMD:D_SMA-SMB_Universal_Handsoldering; LCSC (none) -> C95872; Mfc (none) -> M7
- J5, J6, J7, J8: LCSC (none) -> C8377; Mfc (none) -> WJ2EDGRC-5.08-3P
- K1, K2, K3, K4: LCSC (none) -> C35449; Mfc (none) -> SRD-05VDC-SL-C
- Q1, Q2, Q3, Q4: LCSC (none) -> C75469; Mfc (none) -> FDN340P
- R3, R4, R5, R6: value R -> 10kOhm; LCSC (none) -> C17414; Mfc (none) -> 0805W8F1002T5E
Other:
- moved on the sheet: R3, R4, R5, R6

Commit message: Done PCB Sch Work
Parts:
- J5, J6: footprint (none) -> Connector_Phoenix_MSTB:PhoenixContact_MSTBA_2,5_3-G-5,08_1x03_P5.08mm_Horizontal
- J7, J8: footprint (none) -> Connector_Phoenix_MSTB:PhoenixContact_MSTBVA_2,5_3-G-5,08_1x03_P5.08mm_Vertical; LCSC C8377 -> C8412; Mfc WJ2EDGRC-5.08-3P -> WJ2EDGVC-5.08-3P
- R3, R4, R5, R6: footprint (none) -> Resistor_SMD:R_0805_2012Metric_Pad1.15x1.40mm_HandSolder
Changed lines of the file:
@@
 F 0 "R3" H 2520 1546 50  0000 L CNN
 F 1 "10kOhm" H 2520 1455 50  0000 L CNN
-F 2 "" V 2380 1500 50  0001 C CNN
+F 2 "Resistor_SMD:R_0805_2012Metric_Pad1.15x1.40mm_HandSolder" V 2380 1500 50  0001 C CNN
 F 3 "https://datasheet.lcsc.com/szlcsc/1810271610_UNI-ROYAL-Uniroyal-Elec-0805W8F1002T5E_C17414.pdf" H 2450 1500 50  0001 C CNN
 F 4 "C17414" H 2450 1500 50  0001 C CNN "LCSC"
@@
 F 0 "J5" H 4130 1992 50  0000 L CNN
 F 1 "Screw_Terminal_01x03" H 4130 1901 50  0000 L CNN
-F 2 "" H 4050 1950 50  0001 C CNN
+F 2 "Connector_Phoenix_MSTB:PhoenixContact_MSTBA_2,5_3-G-5,08_1x03_P5.08mm_Horizontal" H 4050 1950 50  0001 C CNN
 F 3 "https://datasheet.lcsc.com/szlcsc/1912251632_Ningbo-Kangnex-Elec-WJ2EDGRC-5-08-3P_C8377.pdf" H 4050 1950 50  0001 C CNN
-F 4 "C8377" H 4050 1950 50  0001 C CNN "LCSC"
+F 4 "C8377" H 4350 2000 50  0000 C CNN "LCSC"
 F 5 "WJ2EDGRC-5.08-3P" H 4050 1950 50  0001 C CNN "Mfc"
 	1    4050 1950
@@
 F 0 "R5" H 7420 1546 50  0000 L CNN
 F 1 "10kOhm" H 7420 1455 50  0000 L CNN
-F 2 "" V 7280 1500 50  0001 C CNN
+F 2 "Resistor_SMD:R_0805_2012Metric_Pad1.15x1.40mm_HandSolder" V 7280 1500 50  0001 C CNN
 F 3 "https://datasheet.lcsc.com/szlcsc/1810271610_UNI-ROYAL-Uniroyal-Elec-0805W8F1002T5E_C17414.pdf" H 7350 1500 50  0001 C CNN
 F 4 "C17414" H 7350 1500 50  0001 C CNN "LCSC"
@@
 F 0 "J7" H 9030 1992 50  0000 L CNN
 F 1 "Screw_Terminal_01x03" H 9030 1901 50  0000 L CNN
-F 2 "" H 8950 1950 50  0001 C CNN
-F 3 "https://datasheet.lcsc.com/szlcsc/1912251632_Ningbo-Kangnex-Elec-WJ2EDGRC-5-08-3P_C8377.pdf" H 8950 1950 50  0001 C CNN
-F 4 "C8377" H 8950 1950 50  0001 C CNN "LCSC"
-F 5 "WJ2EDGRC-5.08-3P" H 8950 1950 50  0001 C CNN "Mfc"
+F 2 "Connector_Phoenix_MSTB:PhoenixContact_MSTBVA_2,5_3-G-5,08_1x03_P5.08mm_Vertical" H 8950 1950 50  0001 C CNN
+F 3 "https://datasheet.lcsc.com/szlcsc/1912251634_Ningbo-Kangnex-Elec-WJ2EDGVC-5-08-3P_C8412.pdf" H 8950 1950 50  0001 C CNN
+F 4 "C8412" H 9250 2000 50  0000 C CNN "LCSC"
+F 5 "WJ2EDGVC-5.08-3P" H 8950 1950 50  0001 C CNN "Mfc"
 	1    8950 1950
 	1    0    0    -1
@@
 F 0 "R4" H 2520 4196 50  0000 L CNN
 F 1 "10kOhm" H 2520 4105 50  0000 L CNN
-F 2 "" V 2380 4150 50  0001 C CNN
+F 2 "Resistor_SMD:R_0805_2012Metric_Pad1.15x1.40mm_HandSolder" V 2380 4150 50  0001 C CNN
 F 3 "https://datasheet.lcsc.com/szlcsc/1810271610_UNI-ROYAL-Uniroyal-Elec-0805W8F1002T5E_C17414.pdf" H 2450 4150 50  0001 C CNN
 F 4 "C17414" H 2450 4150 50  0001 C CNN "LCSC"
@@
 F 0 "J6" H 4130 4642 50  0000 L CNN
 F 1 "Screw_Terminal_01x03" H 4130 4551 50  0000 L CNN
-F 2 "" H 4050 4600 50  0001 C CNN
+F 2 "Connector_Phoenix_MSTB:PhoenixContact_MSTBA_2,5_3-G-5,08_1x03_P5.08mm_Horizontal" H 4050 4600 50  0001 C CNN
 F 3 "https://datasheet.lcsc.com/szlcsc/1912251632_Ningbo-Kangnex-Elec-WJ2EDGRC-5-08-3P_C8377.pdf" H 4050 4600 50  0001 C CNN
-F 4 "C8377" H 4050 4600 50  0001 C CNN "LCSC"
+F 4 "C8377" H 4350 4650 50  0000 C CNN "LCSC"
 F 5 "WJ2EDGRC-5.08-3P" H 4050 4600 50  0001 C CNN "Mfc"
 	1    4050 4600
@@
 F 0 "R6" H 7420 4196 50  0000 L CNN
 F 1 "10kOhm" H 7420 4105 50  0000 L CNN
-F 2 "" V 7280 4150 50  0001 C CNN
+F 2 "Resistor_SMD:R_0805_2012Metric_Pad1.15x1.40mm_HandSolder" V 7280 4150 50  0001 C CNN
 F 3 "https://datasheet.lcsc.com/szlcsc/1810271610_UNI-ROYAL-Uniroyal-Elec-0805W8F1002T5E_C17414.pdf" H 7350 4150 50  0001 C CNN
 F 4 "C17414" H 7350 4150 50  0001 C CNN "LCSC"
@@
 F 0 "J8" H 9030 4642 50  0000 L CNN
 F 1 "Screw_Terminal_01x03" H 9030 4551 50  0000 L CNN
-F 2 "" H 8950 4600 50  0001 C CNN
-F 3 "https://datasheet.lcsc.com/szlcsc/1912251632_Ningbo-Kangnex-Elec-WJ2EDGRC-5-08-3P_C8377.pdf" H 8950 4600 50  0001 C CNN
-F 4 "C8377" H 8950 4600 50  0001 C CNN "LCSC"
-F 5 "WJ2EDGRC-5.08-3P" H 8950 4600 50  0001 C CNN "Mfc"
+F 2 "Connector_Phoenix_MSTB:PhoenixContact_MSTBVA_2,5_3-G-5,08_1x03_P5.08mm_Vertical" H 8950 4600 50  0001 C CNN
+F 3 "https://datasheet.lcsc.com/szlcsc/1912251634_Ningbo-Kangnex-Elec-WJ2EDGVC-5-08-3P_C8412.pdf" H 8950 4600 50  0001 C CNN
+F 4 "C8412" H 9250 4650 50  0000 C CNN "LCSC"
+F 5 "WJ2EDGVC-5.08-3P" H 8950 4600 50  0001 C CNN "Mfc"
 	1    8950 4600
 	1    0    0    -1

Commit message: More PCB Pcb work
Parts:
- C3: symbol Device:CP -> Device:C_Polarized
Changed lines of the file:
@@
 Connection ~ 7350 4500
 $Comp
-L Device:CP C3
+L Device:C_Polarized C3
 U 1 1 5F69DC17
 P 5850 3400
+AR Path="/5F69DC17" Ref="C3"  Part="1"
+AR Path="/5F5F1150/5F5FAAA5/5F69DC17" Ref="C3"  Part="1"
 F 0 "C3" H 5968 3446 50  0000 L CNN
 F 1 "220uF" H 5968 3355 50  0000 L CNN

Commit message: PCB  V1 To production
Parts:
- J7, J8: footprint Connector_Phoenix_MSTB:PhoenixContact_MSTBVA_2,5_3-G-5,08_1x03_P5.08mm_Vertical -> Connector_Phoenix_MSTB:PhoenixContact_MSTBA_2,5_3-G-5,08_1x03_P5.08mm_Horizontal; LCSC C8412 -> C8377; Mfc WJ2EDGVC-5.08-3P -> WJ2EDGRC-5.08-3P
Connections:
- net Output_2: now also Q2.1 (G), R4.2; no longer Q3.1 (G), R5.2
- net Output_3: now also Q3.1 (G), R5.2; no longer Q2.1 (G), R4.2
- net at K3.3: now also J7.1 (Pin_1); no longer J7.3 (Pin_3)
- net at K3.4: now also J7.3 (Pin_3); no longer J7.1 (Pin_1)
- net at K2.3: now also J6.1 (Pin_1); no longer J6.3 (Pin_3)
- net at K2.4: now also J6.3 (Pin_3); no longer J6.1 (Pin_1)
- net at K4.3: now also J8.1 (Pin_1); no longer J8.3 (Pin_3)
- net at K4.4: now also J8.3 (Pin_3); no longer J8.1 (Pin_1)
- net at K1.3: now also J5.1 (Pin_1); no longer J5.3 (Pin_3)
- net at K1.4: now also J5.3 (Pin_3); no longer J5.1 (Pin_1)
Changed lines of the file:
@@
 Wire Wire Line
 	4450 2250 3700 2250
-Wire Wire Line
-	3450 2050 3450 2150
-Wire Wire Line
-	3250 2150 3250 2000
-Wire Wire Line
-	3250 2000 3450 2000
 $Comp
 L Connector:Screw_Terminal_01x03 J5
@@
 Wire Wire Line
 	3700 2250 3700 1950
-Wire Wire Line
-	3450 2050 3850 2050
-Wire Wire Line
-	3450 2000 3450 1850
-Wire Wire Line
-	3450 1850 3850 1850
 Wire Wire Line
 	2350 2300 2350 2100
@@
 	1    0    0    -1
 $EndComp
-Text HLabel 7050 1850 0    50   BiDi ~ 0
+Text HLabel 2150 4500 0    50   BiDi ~ 0
 Output_2
 $Comp
@@
 Wire Wire Line
 	9350 2250 8600 2250
-Wire Wire Line
-	8350 2050 8350 2150
-Wire Wire Line
-	8150 2150 8150 2000
-Wire Wire Line
-	8150 2000 8350 2000
 $Comp
 L Connector:Screw_Terminal_01x03 J7
@@
 F 0 "J7" H 9030 1992 50  0000 L CNN
 F 1 "Screw_Terminal_01x03" H 9030 1901 50  0000 L CNN
-F 2 "Connector_Phoenix_MSTB:PhoenixContact_MSTBVA_2,5_3-G-5,08_1x03_P5.08mm_Vertical" H 8950 1950 50  0001 C CNN
-F 3 "https://datasheet.lcsc.com/szlcsc/1912251634_Ningbo-Kangnex-Elec-WJ2EDGVC-5-08-3P_C8412.pdf" H 8950 1950 50  0001 C CNN
-F 4 "C8412" H 9250 2000 50  0000 C CNN "LCSC"
-F 5 "WJ2EDGVC-5.08-3P" H 8950 1950 50  0001 C CNN "Mfc"
+F 2 "Connector_Phoenix_MSTB:PhoenixContact_MSTBA_2,5_3-G-5,08_1x03_P5.08mm_Horizontal" H 8950 1950 50  0001 C CNN
+F 3 "https://datasheet.lcsc.com/szlcsc/1912251632_Ningbo-Kangnex-Elec-WJ2EDGRC-5-08-3P_C8377.pdf" H 8950 1950 50  0001 C CNN
+F 4 "C8377" H 9250 2000 50  0000 C CNN "LCSC"
+F 5 "WJ2EDGRC-5.08-3P" H 8950 1950 50  0001 C CNN "Mfc"
 	1    8950 1950
 	1    0    0    -1
@@
 Wire Wire Line
 	8600 2250 8600 1950
-Wire Wire Line
-	8350 2050 8750 2050
-Wire Wire Line
-	8350 2000 8350 1850
-Wire Wire Line
-	8350 1850 8750 1850
 Wire Wire Line
 	7250 2300 7250 2100
@@
 	1    0    0    -1
 $EndComp
-Text HLabel 2150 4500 0    50   BiDi ~ 0
+Text HLabel 7050 1850 0    50   BiDi ~ 0
 Output_3
 $Comp
@@
 Wire Wire Line
 	4450 4900 3700 4900
-Wire Wire Line
-	3450 4700 3450 4800
-Wire Wire Line
-	3250 4800 3250 4650
-Wire Wire Line
-	3250 4650 3450 4650
 $Comp
 L Connector:Screw_Terminal_01x03 J6
@@
 Wire Wire Line
 	3700 4900 3700 4600
-Wire Wire Line
-	3450 4700 3850 4700
-Wire Wire Line
-	3450 4650 3450 4500
-Wire Wire Line
-	3450 4500 3850 4500
 Wire Wire Line
 	2350 4950 2350 4750
@@
 Wire Wire Line
 	9350 4900 8600 4900
-Wire Wire Line
-	8350 4700 8350 4800
-Wire Wire Line
-	8150 4800 8150 4650
-Wire Wire Line
-	8150 4650 8350 4650
 $Comp
 L Connector:Screw_Terminal_01x03 J8
@@
 F 0 "J8" H 9030 4642 50  0000 L CNN
 F 1 "Screw_Terminal_01x03" H 9030 4551 50  0000 L CNN
-F 2 "Connector_Phoenix_MSTB:PhoenixContact_MSTBVA_2,5_3-G-5,08_1x03_P5.08mm_Vertical" H 8950 4600 50  0001 C CNN
-F 3 "https://datasheet.lcsc.com/szlcsc/1912251634_Ningbo-Kangnex-Elec-WJ2EDGVC-5-08-3P_C8412.pdf" H 8950 4600 50  0001 C CNN
-F 4 "C8412" H 9250 4650 50  0000 C CNN "LCSC"
-F 5 "WJ2EDGVC-5.08-3P" H 8950 4600 50  0001 C CNN "Mfc"
+F 2 "Connector_Phoenix_MSTB:PhoenixContact_MSTBA_2,5_3-G-5,08_1x03_P5.08mm_Horizontal" H 8950 4600 50  0001 C CNN
+F 3 "https://datasheet.lcsc.com/szlcsc/1912251632_Ningbo-Kangnex-Elec-WJ2EDGRC-5-08-3P_C8377.pdf" H 8950 4600 50  0001 C CNN
+F 4 "C8377" H 9250 4650 50  0000 C CNN "LCSC"
+F 5 "WJ2EDGRC-5.08-3P" H 8950 4600 50  0001 C CNN "Mfc"
 	1    8950 4600
 	1    0    0    -1
@@
 Wire Wire Line
 	8600 4900 8600 4600
-Wire Wire Line
-	8350 4700 8750 4700
-Wire Wire Line
-	8350 4650 8350 4500
-Wire Wire Line
-	8350 4500 8750 4500
 Wire Wire Line
 	7250 4950 7250 4750
@@
 Wire Wire Line
 	5850 3250 5850 3100
+Wire Wire Line
+	8350 1850 8750 1850
+Wire Wire Line
+	8350 1850 8350 2150
+Wire Wire Line
+	8750 2050 8150 2050
+Wire Wire Line
+	8150 2050 8150 2150
+Wire Wire Line
+	8750 4700 8150 4700
+Wire Wire Line
+	8150 4700 8150 4800
+Wire Wire Line
+	8350 4800 8350 4500
+Wire Wire Line
+	8350 4500 8750 4500
+Wire Wire Line
+	3850 4700 3250 4700
+Wire Wire Line
+	3250 4700 3250 4800
+Wire Wire Line
+	3450 4800 3450 4500
+Wire Wire Line
+	3450 4500 3850 4500
+Wire Wire Line
+	3850 2050 3250 2050
+Wire Wire Line
+	3250 2050 3250 2150
+Wire Wire Line
+	3450 2150 3450 1850
+Wire Wire Line
+	3450 1850 3850 1850
 $EndSCHEMATC
