File: Brewnode_PCB/IOExp_Relays.sch (KiCad schematic (older format))
At the start: 21 parts, among them J5 Screw_Terminal_01x03, J6 Screw_Terminal_01x03, J7 Screw_Terminal_01x03, J8 Screw_Terminal_01x03, K1 SANYOU_SRD_Form_C, K2 SANYOU_SRD_Form_C, K3 SANYOU_SRD_Form_C, K4 SANYOU_SRD_Form_C, Q1 FDN340P, Q2 FDN340P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

Commit message: Sch + PCB V1.1
Corrected FDN340 P-FET Pinout.
Added 5V, 3V3 Description in silkscreen for indication D1, D2
Parts:
- C3: symbol Device:C_Polarized -> Brewnode_PCB-rescue:C_Polarized-Device
Connections:
- net +5V: now also Q1.2 (S), Q2.2 (S), Q3.2 (S), Q4.2 (S); no longer Q1.3 (D), Q2.3 (D), Q3.3 (D), Q4.3 (D)
- net at D3.1 (K), K1.5: now also Q1.3 (D); no longer Q1.2 (S)
- net at D5.1 (K), K3.5: now also Q3.3 (D); no longer Q3.2 (S)
- net at D4.1 (K), K2.5: now also Q2.3 (D); no longer Q2.2 (S)
- net at D6.1 (K), K4.5: now also Q4.3 (D); no longer Q4.2 (S)
Changed lines of the file:
@@
 Sheet 4 8
 Title "BrewnodeV1"
-Date "2020-09-16"
-Rev "1.0"
+Date "2020-10-15"
+Rev "1.1"
 Comp "Halldin"
 Comment1 "IOExp_Relays"
@@
 F 5 "FDN340P" H 2850 1850 50  0001 C CNN "Mfc"
 	1    2850 1850
-	1    0    0    -1
+	1    0    0    1
 $EndComp
 $Comp
@@
 	2350 2300 2350 2100
 Wire Wire Line
-	2350 2100 2950 2100
-Wire Wire Line
-	2950 2100 2950 2150
-Wire Wire Line
-	2950 2050 2950 2100
-Connection ~ 2950 2100
-Wire Wire Line
 	2350 2600 2350 2800
 Wire Wire Line
@@
 	2850 1550 2950 1550
 Wire Wire Line
-	2950 1550 2950 1650
-Wire Wire Line
 	2450 1300 2850 1300
 Wire Wire Line
 	2950 1400 2950 1550
-Connection ~ 2950 1550
 Wire Wire Line
 	2450 1650 2450 1850
 Wire Wire Line
-	2450 1850 2650 1850
-Wire Wire Line
 	2450 1850 2150 1850
-Connection ~ 2450 1850
 $Comp
 L Relay:SANYOU_SRD_Form_C K3
@@
 F 5 "FDN340P" H 7750 1850 50  0001 C CNN "Mfc"
 	1    7750 1850
-	1    0    0    -1
+	1    0    0    1
 $EndComp
 $Comp
@@
 	7250 2300 7250 2100
 Wire Wire Line
-	7250 2100 7850 2100
-Wire Wire Line
-	7850 2100 7850 2150
-Wire Wire Line
-	7850 2050 7850 2100
-Connection ~ 7850 2100
-Wire Wire Line
 	7250 2600 7250 2800
 Wire Wire Line
@@
 	7750 1550 7850 1550
 Wire Wire Line
-	7850 1550 7850 1650
-Wire Wire Line
 	7350 1300 7750 1300
 Wire Wire Line
 	7850 1400 7850 1550
-Connection ~ 7850 1550
 Wire Wire Line
 	7350 1650 7350 1850
 Wire Wire Line
-	7350 1850 7550 1850
-Wire Wire Line
 	7350 1850 7050 1850
-Connection ~ 7350 1850
 $Comp
 L Relay:SANYOU_SRD_Form_C K2
@@
 F 5 "FDN340P" H 2850 4500 50  0001 C CNN "Mfc"
 	1    2850 4500
-	1    0    0    -1
+	1    0    0    1
 $EndComp
 $Comp
@@
 	2350 4950 2350 4750
 Wire Wire Line
-	2350 4750 2950 4750
-Wire Wire Line
-	2950 4750 2950 4800
-Wire Wire Line
-	2950 4700 2950 4750
-Connection ~ 2950 4750
-Wire Wire Line
 	2350 5250 2350 5450
 Wire Wire Line
@@
 	2850 4200 2950 4200
 Wire Wire Line
-	2950 4200 2950 4300
-Wire Wire Line
 	2450 3950 2850 3950
 Wire Wire Line
 	2950 4050 2950 4200
-Connection ~ 2950 4200
 Wire Wire Line
 	2450 4300 2450 4500
 Wire Wire Line
-	2450 4500 2650 4500
-Wire Wire Line
 	2450 4500 2150 4500
-Connection ~ 2450 4500
 $Comp
 L Relay:SANYOU_SRD_Form_C K4
@@
 F 5 "FDN340P" H 7750 4500 50  0001 C CNN "Mfc"
 	1    7750 4500
-	1    0    0    -1
+	1    0    0    1
 $EndComp
 $Comp
@@
 	7250 4950 7250 4750
 Wire Wire Line
-	7250 4750 7850 4750
-Wire Wire Line
-	7850 4750 7850 4800
-Wire Wire Line
-	7850 4700 7850 4750
-Connection ~ 7850 4750
-Wire Wire Line
 	7250 5250 7250 5450
 Wire Wire Line
@@
 	7750 4200 7850 4200
 Wire Wire Line
-	7850 4200 7850 4300
-Wire Wire Line
 	7350 3950 7750 3950
 Wire Wire Line
 	7850 4050 7850 4200
-Connection ~ 7850 4200
 Wire Wire Line
 	7350 4300 7350 4500
 Wire Wire Line
-	7350 4500 7550 4500
-Wire Wire Line
 	7350 4500 7050 4500
-Connection ~ 7350 4500
-$Comp
-L Device:C_Polarized C3
+$Comp
+L Brewnode_PCB-rescue:C_Polarized-Device C3
 U 1 1 5F69DC17
 P 5850 3400
@@
 Wire Wire Line
 	3450 1850 3850 1850
+Wire Wire Line
+	2350 2100 2950 2100
+Wire Wire Line
+	2950 2100 2950 2150
+Wire Wire Line
+	2950 2100 2950 2050
+Connection ~ 2950 2100
+Wire Wire Line
+	2450 1850 2650 1850
+Connection ~ 2450 1850
+Wire Wire Line
+	2950 1650 2950 1550
+Connection ~ 2950 1550
+Wire Wire Line
+	7250 2100 7850 2100
+Wire Wire Line
+	7850 2100 7850 2150
+Wire Wire Line
+	7850 2100 7850 2050
+Connection ~ 7850 2100
+Wire Wire Line
+	7350 1850 7550 1850
+Connection ~ 7350 1850
+Wire Wire Line
+	7850 1650 7850 1550
+Connection ~ 7850 1550
+Wire Wire Line
+	7250 4750 7850 4750
+Wire Wire Line
+	7850 4750 7850 4800
+Wire Wire Line
+	7850 4700 7850 4750
+Connection ~ 7850 4750
+Wire Wire Line
+	7350 4500 7550 4500
+Connection ~ 7350 4500
+Wire Wire Line
+	7850 4200 7850 4300
+Connection ~ 7850 4200
+Wire Wire Line
+	2350 4750 2950 4750
+Wire Wire Line
+	2950 4750 2950 4800
+Wire Wire Line
+	2950 4700 2950 4750
+Connection ~ 2950 4750
+Wire Wire Line
+	2450 4500 2650 4500
+Connection ~ 2450 4500
+Wire Wire Line
+	2950 4300 2950 4200
+Connection ~ 2950 4200
 $EndSCHEMATC
