File: Brewnode_PCB/Brewnode_PCB.kicad_pcb (KiCad board)
At the start: 2 copper layers, 83 parts, among them J1 Screw_Terminal_01x03, J10 Screw_Terminal_01x03, J11 Screw_Terminal_01x03, J12 Screw_Terminal_01x03, J13 Screw_Terminal_01x03, J14 Screw_Terminal_01x03, J15 Screw_Terminal_01x03, J16 Screw_Terminal_01x03, J17 16p FPC, J2 Screw_Terminal_01x03, J3 Screw_Terminal_01x03, J4 Screw_Terminal_01x03, J5 Screw_Terminal_01x03, J6 Screw_Terminal_01x03, J7 Screw_Terminal_01x03, J8 Screw_Terminal_01x03, J9 Screw_Terminal_01x03, K1 SANYOU_SRD_Form_C, K2 SANYOU_SRD_Form_C, K3 SANYOU_SRD_Form_C, K4 SANYOU_SRD_Form_C, Q1 FDN340P, Q2 FDN340P, Q3 FDN340P, Q4 FDN340P, Q5 BSS138, Q6 BSS138, Q7 BSS138, Q8 BSS138, U1 PCF8574, U2 ADS1115IDGS

Commit message: PCB  V1 To production
Parts:
- added ?: MountingHole_4mm, MountingHole:MountingHole_4mm, F.Cu at (70.7, 79.9)
- added ?: MountingHole_4mm, MountingHole:MountingHole_4mm, F.Cu at (196.2, 144.3)
- added ?: MountingHole_4mm, MountingHole:MountingHole_4mm, F.Cu at (70.7, 144.3)
- added ?: MountingHole_4mm, MountingHole:MountingHole_4mm, F.Cu at (196.2, 79.9)
- C1, C4, D3, D4, D5, D6, Q5, Q6, Q7, Q8, R10, R11, R12, R13, R14, R15, R16, R17, R18, R19, R20, R21, R22, R23, R24, R25, R26, R27, R28, R29, R30, R7, R8, R9: moved to B.Cu
- J7, J8: footprint Connector_Phoenix_MSTB:PhoenixContact_MSTBVA_2,5_3-G-5,08_1x03_P5.08mm_Vertical -> Connector_Phoenix_MSTB:PhoenixContact_MSTBA_2,5_3-G-5,08_1x03_P5.08mm_Horizontal
- moved U1 145.0 mm to (125.2, 110.6), turned to 270 degrees
- moved D3 129.3 mm to (85.8, 121.3), turned to 180 degrees
- moved C1 127.6 mm to (124.7, 110.6), turned to 90 degrees
- moved J2 118.0 mm to (129.0, 86.4), turned to 180 degrees
- moved R25 112.1 mm to (163.0, 102.5), turned to 90 degrees
- moved R24 110.3 mm to (160.5, 102.5), turned to 90 degrees
- moved R12 106.0 mm to (69.1, 124.1), turned to 180 degrees
- moved R13 104.4 mm to (73.1, 136.3), turned to 180 degrees
- moved JP4 103.4 mm to (69.8, 106.5), turned to 180 degrees
- moved R29 101.5 mm to (126.5, 92.8), turned to 180 degrees
- moved JP1 100.5 mm to (73.6, 91.6)
- moved JP8 99.9 mm to (69.8, 131.2), turned to 180 degrees
- moved R8 99.3 mm to (69.1, 99.2), turned to 180 degrees
- moved R14 99.3 mm to (69.1, 136.3), turned to 180 degrees
- moved Q5 98.1 mm to (141.7, 116.5), turned to 180 degrees
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Connections:
- K1 pad 3: Net-(J5-Pad3) -> Net-(J5-Pad1)
- K1 pad 4: Net-(J5-Pad1) -> Net-(J5-Pad3)
- K2 pad 3: Net-(J6-Pad3) -> Net-(J6-Pad1)
- K2 pad 4: Net-(J6-Pad1) -> Net-(J6-Pad3)
- K3 pad 3: Net-(J7-Pad3) -> Net-(J7-Pad1)
- K3 pad 4: Net-(J7-Pad1) -> Net-(J7-Pad3)
- K4 pad 3: Net-(J8-Pad3) -> Net-(J8-Pad1)
- K4 pad 4: Net-(J8-Pad1) -> Net-(J8-Pad3)
- Q2 pad 1: /IO Expander/IOExp_Relays/Output_3 -> /IO Expander/IOExp_Relays/Output_2
- Q3 pad 1: /IO Expander/IOExp_Relays/Output_2 -> /IO Expander/IOExp_Relays/Output_3
- R23 pad 1: +5V -> +3V3
- R24 pad 1: +5V -> +3V3
- R25 pad 1: +5V -> +3V3
- R26 pad 1: +5V -> +3V3
- R4 pad 2: /IO Expander/IOExp_Relays/Output_3 -> /IO Expander/IOExp_Relays/Output_2
- R5 pad 2: /IO Expander/IOExp_Relays/Output_2 -> /IO Expander/IOExp_Relays/Output_3
Routing:
- net +5V: track 0.00 -> 455.1 mm, vias 0 -> 4
- net GND: track 0.00 -> 181.8 mm, vias 0 -> 20
- net +3V3: track 0.00 -> 105.7 mm, vias 0 -> 7
- net /MCU_Connector/3V3_ADC_Int: track 0.00 -> 78.2 mm, vias 0 -> 3
- net /MCU_Connector/3V3_IOExp_Int: track 0.00 -> 76.1 mm, vias 0 -> 3
- net /ADC/IN_AIN3: track 0.00 -> 67.2 mm, vias 0 -> 1
- net /ADC/5V_ADC_SDA: track 0.00 -> 65.6 mm, vias 0 -> 1
- net /ADC/5V_ADC_SCL: track 0.00 -> 65.1 mm, vias 0 -> 3
- net /ADC/5V_ADC_RDY: track 0.00 -> 61.4 mm, vias 0 -> 3
- net /Digital_Sensors/Port2: track 0.00 -> 59.6 mm
- net /MCU_Connector/3V3_SDA: track 0.00 -> 59.6 mm, vias 0 -> 3
- net /MCU_Connector/3V3_SCL: track 0.00 -> 59.1 mm, vias 0 -> 3
- net /ADC/IN_AIN0: track 0.00 -> 49.2 mm
- net /Digital_Sensors/Port3: track 0.00 -> 46.9 mm
- net Net-(D6-Pad1): track 0.00 -> 46.5 mm, vias 0 -> 1
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- added copper zone on B.Cu, net GND
Other:
- board outline added: 136.9 x 75.8 mm
- rule pad_to_mask_clearance: 0.05 -> 0
- board text added: "10V"
- board text added: "5V"
- board text added: "Brewnode V1"
- board text added: "Port5"
- board text added: "Port6"
- board text added: "Port7"
- board text added: "Port8"

Commit message: Sch + PCB V1.1
Corrected FDN340 P-FET Pinout.
Added 5V, 3V3 Description in silkscreen for indication D1, D2
Connections:
- Q1 pad 2: Net-(D3-Pad1) -> +5V
- Q1 pad 3: +5V -> Net-(D3-Pad1)
- Q2 pad 2: Net-(D4-Pad1) -> +5V
- Q2 pad 3: +5V -> Net-(D4-Pad1)
- Q3 pad 2: Net-(D5-Pad1) -> +5V
- Q3 pad 3: +5V -> Net-(D5-Pad1)
- Q4 pad 2: Net-(D6-Pad1) -> +5V
- Q4 pad 3: +5V -> Net-(D6-Pad1)
Routing:
- net /IO Expander/IOExp_Relays/Output_2: track 10.9 -> 20.2 mm, vias 0 -> 2
- net Net-(D6-Pad1): track 46.5 -> 41.8 mm
- net +5V: track 455.1 -> 459.8 mm
- net Net-(D4-Pad1): track 18.2 -> 13.9 mm
- net Net-(D3-Pad1): track 38.0 -> 35.3 mm
- net /IO Expander/IOExp_Relays/Output_1: track 17.7 -> 19.7 mm
- net /IO Expander/IOExp_Relays/Output_4: track 32.7 -> 34.5 mm, vias 2 -> 3
- net Net-(D5-Pad1): track 25.4 -> 23.8 mm
Other:
- board text added: "3.3V"
- board text added: "Brewnode V1.1"
- board text removed: "Brewnode V1"
