File: Brewnode_PCB/Digital_Sensors.sch (KiCad schematic (older format))
At the start: 9 parts

Commit message: More PCB Sch work
Parts:
- gave numbers to parts that had none: 9
Other:
- moved on the sheet: C6
Changed lines of the file:
@@
 P 8450 3100
 AR Path="/5F5F1150/5F5FA99D/5F673095" Ref="J?"  Part="1"
-AR Path="/5F66FC6A/5F673095" Ref="J?"  Part="1"
-F 0 "J?" H 8530 3142 50  0000 L CNN
+AR Path="/5F66FC6A/5F673095" Ref="J13"  Part="1"
+F 0 "J13" H 8530 3142 50  0000 L CNN
 F 1 "Screw_Terminal_01x03" H 8530 3051 50  0000 L CNN
 F 2 "" H 8450 3100 50  0001 C CNN
@@
 $EndComp
 $Comp
-L power:+5V #PWR?
+L power:+5V #PWR040
 U 1 1 5F6735C9
 P 8000 2750
-F 0 "#PWR?" H 8000 2600 50  0001 C CNN
+F 0 "#PWR040" H 8000 2600 50  0001 C CNN
 F 1 "+5V" H 8015 2923 50  0000 C CNN
 F 2 "" H 8000 2750 50  0001 C CNN
@@
 P 8450 3600
 AR Path="/5F5F1150/5F5FA99D/5F675772" Ref="J?"  Part="1"
-AR Path="/5F66FC6A/5F675772" Ref="J?"  Part="1"
-F 0 "J?" H 8530 3642 50  0000 L CNN
+AR Path="/5F66FC6A/5F675772" Ref="J14"  Part="1"
+F 0 "J14" H 8530 3642 50  0000 L CNN
 F 1 "Screw_Terminal_01x03" H 8530 3551 50  0000 L CNN
 F 2 "" H 8450 3600 50  0001 C CNN
@@
 P 8450 4100
 AR Path="/5F5F1150/5F5FA99D/5F67616B" Ref="J?"  Part="1"
-AR Path="/5F66FC6A/5F67616B" Ref="J?"  Part="1"
-F 0 "J?" H 8530 4142 50  0000 L CNN
+AR Path="/5F66FC6A/5F67616B" Ref="J15"  Part="1"
+F 0 "J15" H 8530 4142 50  0000 L CNN
 F 1 "Screw_Terminal_01x03" H 8530 4051 50  0000 L CNN
 F 2 "" H 8450 4100 50  0001 C CNN
@@
 P 8450 4600
 AR Path="/5F5F1150/5F5FA99D/5F676BDB" Ref="J?"  Part="1"
-AR Path="/5F66FC6A/5F676BDB" Ref="J?"  Part="1"
-F 0 "J?" H 8530 4642 50  0000 L CNN
+AR Path="/5F66FC6A/5F676BDB" Ref="J16"  Part="1"
+F 0 "J16" H 8530 4642 50  0000 L CNN
 F 1 "Screw_Terminal_01x03" H 8530 4551 50  0000 L CNN
 F 2 "" H 8450 4600 50  0001 C CNN
@@
 $EndComp
 $Comp
-L power:GND #PWR?
+L power:GND #PWR041
 U 1 1 5F676D05
 P 8050 5250
-F 0 "#PWR?" H 8050 5000 50  0001 C CNN
+F 0 "#PWR041" H 8050 5000 50  0001 C CNN
 F 1 "GND" H 8055 5077 50  0000 C CNN
 F 2 "" H 8050 5250 50  0001 C CNN
@@
 	8250 3000 8000 3000
 Wire Wire Line
-	8000 3000 8000 2750
+	8000 3000 8000 2800
 Wire Wire Line
 	8250 3500 8000 3500
@@
 Connection ~ 8000 4000
 Wire Wire Line
-	8050 5250 8050 4700
+	8050 5250 8050 5050
 Wire Wire Line
 	8250 4200 8050 4200
@@
 Connection ~ 8050 3700
 $Comp
-L Device:CP C?
+L Device:CP C6
 U 1 1 5F679881
-P 7100 3850
-F 0 "C?" H 7218 3896 50  0000 L CNN
-F 1 "CP" H 7218 3805 50  0000 L CNN
-F 2 "" H 7138 3700 50  0001 C CNN
-F 3 "~" H 7100 3850 50  0001 C CNN
-	1    7100 3850
-	1    0    0    -1
-$EndComp
-Wire Wire Line
-	7100 3700 7100 3000
-Wire Wire Line
-	7100 3000 8000 3000
-Wire Wire Line
-	7100 4000 7100 4700
-Wire Wire Line
-	7100 4700 8050 4700
+P 10000 3800
+F 0 "C6" H 10118 3846 50  0000 L CNN
+F 1 "CP" H 10118 3755 50  0000 L CNN
+F 2 "" H 10038 3650 50  0001 C CNN
+F 3 "~" H 10000 3800 50  0001 C CNN
+	1    10000 3800
+	1    0    0    -1
+$EndComp
 Text HLabel 6650 3100 0    50   BiDi ~ 0
 Port1
@@
 Port4
 $Comp
-L Device:R R?
+L Device:R R23
 U 1 1 5F68371C
 P 6150 2850
-F 0 "R?" H 6220 2896 50  0000 L CNN
+F 0 "R23" H 6220 2896 50  0000 L CNN
 F 1 "4K7" H 6220 2805 50  0000 L CNN
 F 2 "" V 6080 2850 50  0001 C CNN
@@
 $EndComp
 $Comp
-L Device:R R?
+L Device:R R24
 U 1 1 5F684655
 P 6150 3350
-F 0 "R?" H 6220 3396 50  0000 L CNN
+F 0 "R24" H 6220 3396 50  0000 L CNN
 F 1 "4K7" H 6220 3305 50  0000 L CNN
 F 2 "" V 6080 3350 50  0001 C CNN
@@
 $EndComp
 $Comp
-L Device:R R?
+L Device:R R25
 U 1 1 5F6857AA
 P 6150 3850
-F 0 "R?" H 6220 3896 50  0000 L CNN
+F 0 "R25" H 6220 3896 50  0000 L CNN
 F 1 "4K7" H 6220 3805 50  0000 L CNN
 F 2 "" V 6080 3850 50  0001 C CNN
@@
 $EndComp
 $Comp
-L Device:R R?
+L Device:R R26
 U 1 1 5F685F5C
 P 6150 4350
-F 0 "R?" H 6220 4396 50  0000 L CNN
+F 0 "R26" H 6220 4396 50  0000 L CNN
 F 1 "4K7" H 6220 4305 50  0000 L CNN
 F 2 "" V 6080 4350 50  0001 C CNN
@@
 $EndComp
 $Comp
-L power:+5V #PWR?
+L power:+5V #PWR039
 U 1 1 5F688119
 P 6000 2600
-F 0 "#PWR?" H 6000 2450 50  0001 C CNN
+F 0 "#PWR039" H 6000 2450 50  0001 C CNN
 F 1 "+5V" H 6015 2773 50  0000 C CNN
 F 2 "" H 6000 2600 50  0001 C CNN
@@
 Wire Wire Line
 	6900 4600 8250 4600
+Wire Wire Line
+	10000 3650 10000 2800
+Wire Wire Line
+	10000 2800 8000 2800
+Connection ~ 8000 2800
+Wire Wire Line
+	8000 2800 8000 2750
+Wire Wire Line
+	10000 3950 10000 5050
+Wire Wire Line
+	10000 5050 8050 5050
+Connection ~ 8050 5050
+Wire Wire Line
+	8050 5050 8050 4700
 $EndSCHEMATC

Commit message: More PCB Sch work
Parts:
- C6: value CP -> 47uF; footprint (none) -> Capacitor_SMD:CP_Elec_6.3x5.3; LCSC (none) -> C249778; Mfc (none) -> VEZ470M1CTR-0605
- J13, J14, J15, J16: LCSC (none) -> C8377; Mfc (none) -> WJ2EDGRC-5.08-3P
- R23, R24, R25, R26: value 4K7 -> 4.7kOhm; LCSC (none) -> C17673; Mfc (none) -> 0805W8F4701T5E
Changed lines of the file:
@@
 F 1 "Screw_Terminal_01x03" H 8530 3051 50  0000 L CNN
 F 2 "" H 8450 3100 50  0001 C CNN
-F 3 "~" H 8450 3100 50  0001 C CNN
+F 3 "https://datasheet.lcsc.com/szlcsc/1912251632_Ningbo-Kangnex-Elec-WJ2EDGRC-5-08-3P_C8377.pdf" H 8450 3100 50  0001 C CNN
+F 4 "C8377" H 8450 3100 50  0001 C CNN "LCSC"
+F 5 "WJ2EDGRC-5.08-3P" H 8450 3100 50  0001 C CNN "Mfc"
 	1    8450 3100
 	1    0    0    -1
@@
 F 1 "Screw_Terminal_01x03" H 8530 3551 50  0000 L CNN
 F 2 "" H 8450 3600 50  0001 C CNN
-F 3 "~" H 8450 3600 50  0001 C CNN
+F 3 "https://datasheet.lcsc.com/szlcsc/1912251632_Ningbo-Kangnex-Elec-WJ2EDGRC-5-08-3P_C8377.pdf" H 8450 3600 50  0001 C CNN
+F 4 "C8377" H 8450 3600 50  0001 C CNN "LCSC"
+F 5 "WJ2EDGRC-5.08-3P" H 8450 3600 50  0001 C CNN "Mfc"
 	1    8450 3600
 	1    0    0    -1
@@
 F 1 "Screw_Terminal_01x03" H 8530 4051 50  0000 L CNN
 F 2 "" H 8450 4100 50  0001 C CNN
-F 3 "~" H 8450 4100 50  0001 C CNN
+F 3 "https://datasheet.lcsc.com/szlcsc/1912251632_Ningbo-Kangnex-Elec-WJ2EDGRC-5-08-3P_C8377.pdf" H 8450 4100 50  0001 C CNN
+F 4 "C8377" H 8450 4100 50  0001 C CNN "LCSC"
+F 5 "WJ2EDGRC-5.08-3P" H 8450 4100 50  0001 C CNN "Mfc"
 	1    8450 4100
 	1    0    0    -1
@@
 F 1 "Screw_Terminal_01x03" H 8530 4551 50  0000 L CNN
 F 2 "" H 8450 4600 50  0001 C CNN
-F 3 "~" H 8450 4600 50  0001 C CNN
+F 3 "https://datasheet.lcsc.com/szlcsc/1912251632_Ningbo-Kangnex-Elec-WJ2EDGRC-5-08-3P_C8377.pdf" H 8450 4600 50  0001 C CNN
+F 4 "C8377" H 8450 4600 50  0001 C CNN "LCSC"
+F 5 "WJ2EDGRC-5.08-3P" H 8450 4600 50  0001 C CNN "Mfc"
 	1    8450 4600
 	1    0    0    -1
@@
 P 10000 3800
 F 0 "C6" H 10118 3846 50  0000 L CNN
-F 1 "CP" H 10118 3755 50  0000 L CNN
-F 2 "" H 10038 3650 50  0001 C CNN
-F 3 "~" H 10000 3800 50  0001 C CNN
+F 1 "47uF" H 10118 3755 50  0000 L CNN
+F 2 "Capacitor_SMD:CP_Elec_6.3x5.3" H 10038 3650 50  0001 C CNN
+F 3 "https://datasheet.lcsc.com/szlcsc/1912111437_Lelon-VEZ470M1CTR-0605_C249778.pdf" H 10000 3800 50  0001 C CNN
+F 4 "C249778" H 10000 3800 50  0001 C CNN "LCSC"
+F 5 "	VEZ470M1CTR-0605" H 10000 3800 50  0001 C CNN "Mfc"
 	1    10000 3800
 	1    0    0    -1
@@
 P 6150 2850
 F 0 "R23" H 6220 2896 50  0000 L CNN
-F 1 "4K7" H 6220 2805 50  0000 L CNN
+F 1 "4.7kOhm" H 6220 2805 50  0000 L CNN
 F 2 "" V 6080 2850 50  0001 C CNN
-F 3 "~" H 6150 2850 50  0001 C CNN
+F 3 "https://datasheet.lcsc.com/szlcsc/1808281533_UNI-ROYAL-Uniroyal-Elec-0805W8F4701T5E_C17673.pdf" H 6150 2850 50  0001 C CNN
+F 4 "C17673" H 6150 2850 50  0001 C CNN "LCSC"
+F 5 "0805W8F4701T5E" H 6150 2850 50  0001 C CNN "Mfc"
 	1    6150 2850
 	1    0    0    -1
@@
 P 6150 3350
 F 0 "R24" H 6220 3396 50  0000 L CNN
-F 1 "4K7" H 6220 3305 50  0000 L CNN
+F 1 "4.7kOhm" H 6220 3305 50  0000 L CNN
 F 2 "" V 6080 3350 50  0001 C CNN
-F 3 "~" H 6150 3350 50  0001 C CNN
+F 3 "https://datasheet.lcsc.com/szlcsc/1808281533_UNI-ROYAL-Uniroyal-Elec-0805W8F4701T5E_C17673.pdf" H 6150 3350 50  0001 C CNN
+F 4 "C17673" H 6150 3350 50  0001 C CNN "LCSC"
+F 5 "0805W8F4701T5E" H 6150 3350 50  0001 C CNN "Mfc"
 	1    6150 3350
 	1    0    0    -1
@@
 P 6150 3850
 F 0 "R25" H 6220 3896 50  0000 L CNN
-F 1 "4K7" H 6220 3805 50  0000 L CNN
+F 1 "4.7kOhm" H 6220 3805 50  0000 L CNN
 F 2 "" V 6080 3850 50  0001 C CNN
-F 3 "~" H 6150 3850 50  0001 C CNN
+F 3 "https://datasheet.lcsc.com/szlcsc/1808281533_UNI-ROYAL-Uniroyal-Elec-0805W8F4701T5E_C17673.pdf" H 6150 3850 50  0001 C CNN
+F 4 "C17673" H 6150 3850 50  0001 C CNN "LCSC"
+F 5 "0805W8F4701T5E" H 6150 3850 50  0001 C CNN "Mfc"
 	1    6150 3850
 	1    0    0    -1
@@
 P 6150 4350
 F 0 "R26" H 6220 4396 50  0000 L CNN
-F 1 "4K7" H 6220 4305 50  0000 L CNN
+F 1 "4.7kOhm" H 6220 4305 50  0000 L CNN
 F 2 "" V 6080 4350 50  0001 C CNN
-F 3 "~" H 6150 4350 50  0001 C CNN
+F 3 "https://datasheet.lcsc.com/szlcsc/1808281533_UNI-ROYAL-Uniroyal-Elec-0805W8F4701T5E_C17673.pdf" H 6150 4350 50  0001 C CNN
+F 4 "C17673" H 6150 4350 50  0001 C CNN "LCSC"
+F 5 "0805W8F4701T5E" H 6150 4350 50  0001 C CNN "Mfc"
 	1    6150 4350
 	1    0    0    -1

Commit message: Done PCB Sch Work
Parts:
- J13, J14: footprint (none) -> Connector_Phoenix_MSTB:PhoenixContact_MSTBA_2,5_3-G-5,08_1x03_P5.08mm_Horizontal
- J15, J16: footprint (none) -> Connector_Phoenix_MSTB:PhoenixContact_MSTBVA_2,5_3-G-5,08_1x03_P5.08mm_Vertical; LCSC C8377 -> C8412; Mfc WJ2EDGRC-5.08-3P -> WJ2EDGVC-5.08-3P
- R23, R24, R25, R26: footprint (none) -> Resistor_SMD:R_0805_2012Metric_Pad1.15x1.40mm_HandSolder
Changed lines of the file:
@@
 F 0 "J13" H 8530 3142 50  0000 L CNN
 F 1 "Screw_Terminal_01x03" H 8530 3051 50  0000 L CNN
-F 2 "" H 8450 3100 50  0001 C CNN
+F 2 "Connector_Phoenix_MSTB:PhoenixContact_MSTBA_2,5_3-G-5,08_1x03_P5.08mm_Horizontal" H 8450 3100 50  0001 C CNN
 F 3 "https://datasheet.lcsc.com/szlcsc/1912251632_Ningbo-Kangnex-Elec-WJ2EDGRC-5-08-3P_C8377.pdf" H 8450 3100 50  0001 C CNN
-F 4 "C8377" H 8450 3100 50  0001 C CNN "LCSC"
+F 4 "C8377" H 8800 3150 50  0000 C CNN "LCSC"
 F 5 "WJ2EDGRC-5.08-3P" H 8450 3100 50  0001 C CNN "Mfc"
 	1    8450 3100
@@
 F 0 "J14" H 8530 3642 50  0000 L CNN
 F 1 "Screw_Terminal_01x03" H 8530 3551 50  0000 L CNN
-F 2 "" H 8450 3600 50  0001 C CNN
+F 2 "Connector_Phoenix_MSTB:PhoenixContact_MSTBA_2,5_3-G-5,08_1x03_P5.08mm_Horizontal" H 8450 3600 50  0001 C CNN
 F 3 "https://datasheet.lcsc.com/szlcsc/1912251632_Ningbo-Kangnex-Elec-WJ2EDGRC-5-08-3P_C8377.pdf" H 8450 3600 50  0001 C CNN
-F 4 "C8377" H 8450 3600 50  0001 C CNN "LCSC"
+F 4 "C8377" H 8800 3650 50  0000 C CNN "LCSC"
 F 5 "WJ2EDGRC-5.08-3P" H 8450 3600 50  0001 C CNN "Mfc"
 	1    8450 3600
@@
 F 0 "J15" H 8530 4142 50  0000 L CNN
 F 1 "Screw_Terminal_01x03" H 8530 4051 50  0000 L CNN
-F 2 "" H 8450 4100 50  0001 C CNN
-F 3 "https://datasheet.lcsc.com/szlcsc/1912251632_Ningbo-Kangnex-Elec-WJ2EDGRC-5-08-3P_C8377.pdf" H 8450 4100 50  0001 C CNN
-F 4 "C8377" H 8450 4100 50  0001 C CNN "LCSC"
-F 5 "WJ2EDGRC-5.08-3P" H 8450 4100 50  0001 C CNN "Mfc"
+F 2 "Connector_Phoenix_MSTB:PhoenixContact_MSTBVA_2,5_3-G-5,08_1x03_P5.08mm_Vertical" H 8450 4100 50  0001 C CNN
+F 3 "https://datasheet.lcsc.com/szlcsc/1912251634_Ningbo-Kangnex-Elec-WJ2EDGVC-5-08-3P_C8412.pdf" H 8450 4100 50  0001 C CNN
+F 4 "C8412" H 8800 4150 50  0000 C CNN "LCSC"
+F 5 "WJ2EDGVC-5.08-3P" H 8450 4100 50  0001 C CNN "Mfc"
 	1    8450 4100
 	1    0    0    -1
@@
 F 0 "J16" H 8530 4642 50  0000 L CNN
 F 1 "Screw_Terminal_01x03" H 8530 4551 50  0000 L CNN
-F 2 "" H 8450 4600 50  0001 C CNN
-F 3 "https://datasheet.lcsc.com/szlcsc/1912251632_Ningbo-Kangnex-Elec-WJ2EDGRC-5-08-3P_C8377.pdf" H 8450 4600 50  0001 C CNN
-F 4 "C8377" H 8450 4600 50  0001 C CNN "LCSC"
-F 5 "WJ2EDGRC-5.08-3P" H 8450 4600 50  0001 C CNN "Mfc"
+F 2 "Connector_Phoenix_MSTB:PhoenixContact_MSTBVA_2,5_3-G-5,08_1x03_P5.08mm_Vertical" H 8450 4600 50  0001 C CNN
+F 3 "https://datasheet.lcsc.com/szlcsc/1912251634_Ningbo-Kangnex-Elec-WJ2EDGVC-5-08-3P_C8412.pdf" H 8450 4600 50  0001 C CNN
+F 4 "C8412" H 8800 4650 50  0000 C CNN "LCSC"
+F 5 "WJ2EDGVC-5.08-3P" H 8450 4600 50  0001 C CNN "Mfc"
 	1    8450 4600
 	1    0    0    -1
@@
 F 0 "R23" H 6220 2896 50  0000 L CNN
 F 1 "4.7kOhm" H 6220 2805 50  0000 L CNN
-F 2 "" V 6080 2850 50  0001 C CNN
+F 2 "Resistor_SMD:R_0805_2012Metric_Pad1.15x1.40mm_HandSolder" V 6080 2850 50  0001 C CNN
 F 3 "https://datasheet.lcsc.com/szlcsc/1808281533_UNI-ROYAL-Uniroyal-Elec-0805W8F4701T5E_C17673.pdf" H 6150 2850 50  0001 C CNN
 F 4 "C17673" H 6150 2850 50  0001 C CNN "LCSC"
@@
 F 0 "R24" H 6220 3396 50  0000 L CNN
 F 1 "4.7kOhm" H 6220 3305 50  0000 L CNN
-F 2 "" V 6080 3350 50  0001 C CNN
+F 2 "Resistor_SMD:R_0805_2012Metric_Pad1.15x1.40mm_HandSolder" V 6080 3350 50  0001 C CNN
 F 3 "https://datasheet.lcsc.com/szlcsc/1808281533_UNI-ROYAL-Uniroyal-Elec-0805W8F4701T5E_C17673.pdf" H 6150 3350 50  0001 C CNN
 F 4 "C17673" H 6150 3350 50  0001 C CNN "LCSC"
@@
 F 0 "R25" H 6220 3896 50  0000 L CNN
 F 1 "4.7kOhm" H 6220 3805 50  0000 L CNN
-F 2 "" V 6080 3850 50  0001 C CNN
+F 2 "Resistor_SMD:R_0805_2012Metric_Pad1.15x1.40mm_HandSolder" V 6080 3850 50  0001 C CNN
 F 3 "https://datasheet.lcsc.com/szlcsc/1808281533_UNI-ROYAL-Uniroyal-Elec-0805W8F4701T5E_C17673.pdf" H 6150 3850 50  0001 C CNN
 F 4 "C17673" H 6150 3850 50  0001 C CNN "LCSC"
@@
 F 0 "R26" H 6220 4396 50  0000 L CNN
 F 1 "4.7kOhm" H 6220 4305 50  0000 L CNN
-F 2 "" V 6080 4350 50  0001 C CNN
+F 2 "Resistor_SMD:R_0805_2012Metric_Pad1.15x1.40mm_HandSolder" V 6080 4350 50  0001 C CNN
 F 3 "https://datasheet.lcsc.com/szlcsc/1808281533_UNI-ROYAL-Uniroyal-Elec-0805W8F4701T5E_C17673.pdf" H 6150 4350 50  0001 C CNN
 F 4 "C17673" H 6150 4350 50  0001 C CNN "LCSC"

Commit message: More PCB Pcb work
Parts:
- C6: symbol Device:CP -> Device:C_Polarized
Changed lines of the file:
@@
 Connection ~ 8050 3700
 $Comp
-L Device:CP C6
+L Device:C_Polarized C6
 U 1 1 5F679881
 P 10000 3800
+AR Path="/5F679881" Ref="C6"  Part="1"
+AR Path="/5F66FC6A/5F679881" Ref="C6"  Part="1"
 F 0 "C6" H 10118 3846 50  0000 L CNN
 F 1 "47uF" H 10118 3755 50  0000 L CNN

Commit message: PCB  V1 To production
Connections:
- net +5V: no longer R23.1, R24.1, R25.1, R26.1
- new net +3V3: R23.1, R24.1, R25.1, R26.1
Changed lines of the file:
@@
-	1    0    0    -1
-$EndComp
-$Comp
-L power:+5V #PWR039
-U 1 1 5F688119
-P 6000 2600
-F 0 "#PWR039" H 6000 2450 50  0001 C CNN
-F 1 "+5V" H 6015 2773 50  0000 C CNN
-F 2 "" H 6000 2600 50  0001 C CNN
-F 3 "" H 6000 2600 50  0001 C CNN
-	1    6000 2600
 	1    0    0    -1
 $EndComp
@@
 Wire Wire Line
 	8050 5050 8050 4700
+$Comp
+L power:+3V3 #PWR0101
+U 1 1 5F6B554D
+P 6000 2600
+F 0 "#PWR0101" H 6000 2450 50  0001 C CNN
+F 1 "+3V3" H 6015 2773 50  0000 C CNN
+F 2 "" H 6000 2600 50  0001 C CNN
+F 3 "" H 6000 2600 50  0001 C CNN
+	1    6000 2600
+	1    0    0    -1
+$EndComp
 $EndSCHEMATC

Commit message: Sch + PCB V1.1
Corrected FDN340 P-FET Pinout.
Added 5V, 3V3 Description in silkscreen for indication D1, D2
Parts:
- C6: symbol Device:C_Polarized -> Brewnode_PCB-rescue:C_Polarized-Device
Changed lines of the file:
@@
 Sheet 7 8
 Title "BrewnodeV1"
-Date "2020-09-16"
-Rev "1.0"
+Date "2020-10-15"
+Rev "1.1"
 Comp "Halldin"
 Comment1 "Digital Sensors"
@@
 Connection ~ 8050 3700
 $Comp
-L Device:C_Polarized C6
+L Brewnode_PCB-rescue:C_Polarized-Device C6
 U 1 1 5F679881
 P 10000 3800
