File: Brewnode_PCB/Lvl_Shifter.sch (KiCad schematic (older format))
At the start: 12 parts

Commit message: More PCB Sch work
Parts:
- gave numbers to parts that had none: 12
Changed lines of the file:
@@
 HV_4
 $Comp
-L Transistor_FET:BSS138 Q?
+L Transistor_FET:BSS138 Q5
 U 1 1 5F616C31
 P 4000 2400
-F 0 "Q?" V 4249 2400 50  0000 C CNN
+F 0 "Q5" V 4249 2400 50  0000 C CNN
 F 1 "BSS138" V 4340 2400 50  0000 C CNN
 F 2 "Package_TO_SOT_SMD:SOT-23" H 4200 2325 50  0001 L CIN
@@
 $EndComp
 $Comp
-L Transistor_FET:BSS138 Q?
+L Transistor_FET:BSS138 Q6
 U 1 1 5F61F40A
 P 4000 3400
-F 0 "Q?" V 4249 3400 50  0000 C CNN
+F 0 "Q6" V 4249 3400 50  0000 C CNN
 F 1 "BSS138" V 4340 3400 50  0000 C CNN
 F 2 "Package_TO_SOT_SMD:SOT-23" H 4200 3325 50  0001 L CIN
@@
 $EndComp
 $Comp
-L Transistor_FET:BSS138 Q?
+L Transistor_FET:BSS138 Q7
 U 1 1 5F6211B8
 P 4000 4400
-F 0 "Q?" V 4249 4400 50  0000 C CNN
+F 0 "Q7" V 4249 4400 50  0000 C CNN
 F 1 "BSS138" V 4340 4400 50  0000 C CNN
 F 2 "Package_TO_SOT_SMD:SOT-23" H 4200 4325 50  0001 L CIN
@@
 $EndComp
 $Comp
-L Transistor_FET:BSS138 Q?
+L Transistor_FET:BSS138 Q8
 U 1 1 5F622813
 P 4000 5400
-F 0 "Q?" V 4249 5400 50  0000 C CNN
+F 0 "Q8" V 4249 5400 50  0000 C CNN
 F 1 "BSS138" V 4340 5400 50  0000 C CNN
 F 2 "Package_TO_SOT_SMD:SOT-23" H 4200 5325 50  0001 L CIN
@@
 $EndComp
 $Comp
-L Device:R R?
+L Device:R R15
 U 1 1 5F628659
 P 3000 2350
-F 0 "R?" H 3070 2396 50  0000 L CNN
+F 0 "R15" H 3070 2396 50  0000 L CNN
 F 1 "10K" H 3070 2305 50  0000 L CNN
 F 2 "" V 2930 2350 50  0001 C CNN
@@
 $EndComp
 $Comp
-L Device:R R?
+L Device:R R16
 U 1 1 5F62A38F
 P 3000 3350
-F 0 "R?" H 3070 3396 50  0000 L CNN
+F 0 "R16" H 3070 3396 50  0000 L CNN
 F 1 "10K" H 3070 3305 50  0000 L CNN
 F 2 "" V 2930 3350 50  0001 C CNN
@@
 $EndComp
 $Comp
-L Device:R R?
+L Device:R R18
 U 1 1 5F62D0C7
 P 3000 5350
-F 0 "R?" H 3070 5396 50  0000 L CNN
+F 0 "R18" H 3070 5396 50  0000 L CNN
 F 1 "10K" H 3070 5305 50  0000 L CNN
 F 2 "" V 2930 5350 50  0001 C CNN
@@
 $EndComp
 $Comp
-L Device:R R?
+L Device:R R22
 U 1 1 5F62D0CD
 P 5000 5350
-F 0 "R?" H 5070 5396 50  0000 L CNN
+F 0 "R22" H 5070 5396 50  0000 L CNN
 F 1 "10K" H 5070 5305 50  0000 L CNN
 F 2 "" V 4930 5350 50  0001 C CNN
@@
 $EndComp
 $Comp
-L Device:R R?
+L Device:R R17
 U 1 1 5F62DDE3
 P 3000 4350
-F 0 "R?" H 3070 4396 50  0000 L CNN
+F 0 "R17" H 3070 4396 50  0000 L CNN
 F 1 "10K" H 3070 4305 50  0000 L CNN
 F 2 "" V 2930 4350 50  0001 C CNN
@@
 $EndComp
 $Comp
-L Device:R R?
+L Device:R R21
 U 1 1 5F62DDE9
 P 5000 4350
-F 0 "R?" H 5070 4396 50  0000 L CNN
+F 0 "R21" H 5070 4396 50  0000 L CNN
 F 1 "10K" H 5070 4305 50  0000 L CNN
 F 2 "" V 4930 4350 50  0001 C CNN
@@
 $EndComp
 $Comp
-L Device:R R?
+L Device:R R19
 U 1 1 5F62E36B
 P 5000 2350
-F 0 "R?" H 5070 2396 50  0000 L CNN
+F 0 "R19" H 5070 2396 50  0000 L CNN
 F 1 "10K" H 5070 2305 50  0000 L CNN
 F 2 "" V 4930 2350 50  0001 C CNN
@@
 $EndComp
 $Comp
-L Device:R R?
+L Device:R R20
 U 1 1 5F62E371
 P 5000 3350
-F 0 "R?" H 5070 3396 50  0000 L CNN
+F 0 "R20" H 5070 3396 50  0000 L CNN
 F 1 "10K" H 5070 3305 50  0000 L CNN
 F 2 "" V 4930 3350 50  0001 C CNN
@@
 $EndComp
 $Comp
-L power:+3V3 #PWR?
+L power:+3V3 #PWR031
 U 1 1 5F653492
 P 4000 2100
-F 0 "#PWR?" H 4000 1950 50  0001 C CNN
+F 0 "#PWR031" H 4000 1950 50  0001 C CNN
 F 1 "+3V3" H 4015 2273 50  0000 C CNN
 F 2 "" H 4000 2100 50  0001 C CNN
@@
 $EndComp
 $Comp
-L power:+5V #PWR?
+L power:+5V #PWR035
 U 1 1 5F6546A0
 P 5000 2100
-F 0 "#PWR?" H 5000 1950 50  0001 C CNN
+F 0 "#PWR035" H 5000 1950 50  0001 C CNN
 F 1 "+5V" H 5015 2273 50  0000 C CNN
 F 2 "" H 5000 2100 50  0001 C CNN
@@
 $EndComp
 $Comp
-L power:+3V3 #PWR?
+L power:+3V3 #PWR032
 U 1 1 5F6560FA
 P 4000 3100
-F 0 "#PWR?" H 4000 2950 50  0001 C CNN
+F 0 "#PWR032" H 4000 2950 50  0001 C CNN
 F 1 "+3V3" H 4015 3273 50  0000 C CNN
 F 2 "" H 4000 3100 50  0001 C CNN
@@
 $EndComp
 $Comp
-L power:+3V3 #PWR?
+L power:+3V3 #PWR027
 U 1 1 5F656D5E
 P 3000 2100
-F 0 "#PWR?" H 3000 1950 50  0001 C CNN
+F 0 "#PWR027" H 3000 1950 50  0001 C CNN
 F 1 "+3V3" H 3015 2273 50  0000 C CNN
 F 2 "" H 3000 2100 50  0001 C CNN
@@
 $EndComp
 $Comp
-L power:+3V3 #PWR?
+L power:+3V3 #PWR028
 U 1 1 5F657130
 P 3000 3100
-F 0 "#PWR?" H 3000 2950 50  0001 C CNN
+F 0 "#PWR028" H 3000 2950 50  0001 C CNN
 F 1 "+3V3" H 3015 3273 50  0000 C CNN
 F 2 "" H 3000 3100 50  0001 C CNN
@@
 $EndComp
 $Comp
-L power:+3V3 #PWR?
+L power:+3V3 #PWR033
 U 1 1 5F65A9C9
 P 4000 4100
-F 0 "#PWR?" H 4000 3950 50  0001 C CNN
+F 0 "#PWR033" H 4000 3950 50  0001 C CNN
 F 1 "+3V3" H 4015 4273 50  0000 C CNN
 F 2 "" H 4000 4100 50  0001 C CNN
@@
 $EndComp
 $Comp
-L power:+3V3 #PWR?
+L power:+3V3 #PWR029
 U 1 1 5F65AB88
 P 3000 4100
-F 0 "#PWR?" H 3000 3950 50  0001 C CNN
+F 0 "#PWR029" H 3000 3950 50  0001 C CNN
 F 1 "+3V3" H 3015 4273 50  0000 C CNN
 F 2 "" H 3000 4100 50  0001 C CNN
@@
 $EndComp
 $Comp
-L power:+3V3 #PWR?
+L power:+3V3 #PWR030
 U 1 1 5F65DC0D
 P 3000 5100
-F 0 "#PWR?" H 3000 4950 50  0001 C CNN
+F 0 "#PWR030" H 3000 4950 50  0001 C CNN
 F 1 "+3V3" H 3015 5273 50  0000 C CNN
 F 2 "" H 3000 5100 50  0001 C CNN
@@
 $EndComp
 $Comp
-L power:+3V3 #PWR?
+L power:+3V3 #PWR034
 U 1 1 5F65DF34
 P 4000 5100
-F 0 "#PWR?" H 4000 4950 50  0001 C CNN
+F 0 "#PWR034" H 4000 4950 50  0001 C CNN
 F 1 "+3V3" H 4015 5273 50  0000 C CNN
 F 2 "" H 4000 5100 50  0001 C CNN
@@
 $EndComp
 $Comp
-L power:+5V #PWR?
+L power:+5V #PWR036
 U 1 1 5F66543D
 P 5000 3100
-F 0 "#PWR?" H 5000 2950 50  0001 C CNN
+F 0 "#PWR036" H 5000 2950 50  0001 C CNN
 F 1 "+5V" H 5015 3273 50  0000 C CNN
 F 2 "" H 5000 3100 50  0001 C CNN
@@
 $EndComp
 $Comp
-L power:+5V #PWR?
+L power:+5V #PWR037
 U 1 1 5F6656D7
 P 5000 4100
-F 0 "#PWR?" H 5000 3950 50  0001 C CNN
+F 0 "#PWR037" H 5000 3950 50  0001 C CNN
 F 1 "+5V" H 5015 4273 50  0000 C CNN
 F 2 "" H 5000 4100 50  0001 C CNN
@@
 $EndComp
 $Comp
-L power:+5V #PWR?
+L power:+5V #PWR038
 U 1 1 5F66583B
 P 5000 5100
-F 0 "#PWR?" H 5000 4950 50  0001 C CNN
+F 0 "#PWR038" H 5000 4950 50  0001 C CNN
 F 1 "+5V" H 5015 5273 50  0000 C CNN
 F 2 "" H 5000 5100 50  0001 C CNN

Commit message: More PCB Sch work
Parts:
- Q5, Q6, Q7, Q8: LCSC (none) -> C52895; Mfc (none) -> BSS138
- R15, R16, R17, R18, R19, R20, R21, R22: value 10K -> 10kOhm; LCSC (none) -> C17414; Mfc (none) -> 0805W8F1000T5E
Changed lines of the file:
@@
 F 2 "Package_TO_SOT_SMD:SOT-23" H 4200 2325 50  0001 L CIN
 F 3 "https://www.onsemi.com/pub/Collateral/BSS138-D.PDF" H 4000 2400 50  0001 L CNN
+F 4 "C52895" H 4000 2400 50  0001 C CNN "LCSC"
+F 5 "BSS138" H 4000 2400 50  0001 C CNN "Mfc"
 	1    4000 2400
 	0    1    1    0
@@
 F 2 "Package_TO_SOT_SMD:SOT-23" H 4200 3325 50  0001 L CIN
 F 3 "https://www.onsemi.com/pub/Collateral/BSS138-D.PDF" H 4000 3400 50  0001 L CNN
+F 4 "C52895" H 4000 3400 50  0001 C CNN "LCSC"
+F 5 "BSS138" H 4000 3400 50  0001 C CNN "Mfc"
 	1    4000 3400
 	0    1    1    0
@@
 F 2 "Package_TO_SOT_SMD:SOT-23" H 4200 4325 50  0001 L CIN
 F 3 "https://www.onsemi.com/pub/Collateral/BSS138-D.PDF" H 4000 4400 50  0001 L CNN
+F 4 "C52895" H 4000 4400 50  0001 C CNN "LCSC"
+F 5 "BSS138" H 4000 4400 50  0001 C CNN "Mfc"
 	1    4000 4400
 	0    1    1    0
@@
 F 2 "Package_TO_SOT_SMD:SOT-23" H 4200 5325 50  0001 L CIN
 F 3 "https://www.onsemi.com/pub/Collateral/BSS138-D.PDF" H 4000 5400 50  0001 L CNN
+F 4 "C52895" H 4000 5400 50  0001 C CNN "LCSC"
+F 5 "BSS138" H 4000 5400 50  0001 C CNN "Mfc"
 	1    4000 5400
 	0    1    1    0
@@
 P 3000 2350
 F 0 "R15" H 3070 2396 50  0000 L CNN
-F 1 "10K" H 3070 2305 50  0000 L CNN
+F 1 "10kOhm" H 3070 2305 50  0000 L CNN
 F 2 "" V 2930 2350 50  0001 C CNN
-F 3 "~" H 3000 2350 50  0001 C CNN
+F 3 "https://datasheet.lcsc.com/szlcsc/1810271610_UNI-ROYAL-Uniroyal-Elec-0805W8F1002T5E_C17414.pdf" H 3000 2350 50  0001 C CNN
+F 4 "C17414" H 3000 2350 50  0001 C CNN "LCSC"
+F 5 "0805W8F1000T5E" H 3000 2350 50  0001 C CNN "Mfc"
 	1    3000 2350
 	1    0    0    -1
@@
 P 3000 3350
 F 0 "R16" H 3070 3396 50  0000 L CNN
-F 1 "10K" H 3070 3305 50  0000 L CNN
+F 1 "10kOhm" H 3070 3305 50  0000 L CNN
 F 2 "" V 2930 3350 50  0001 C CNN
-F 3 "~" H 3000 3350 50  0001 C CNN
+F 3 "https://datasheet.lcsc.com/szlcsc/1810271610_UNI-ROYAL-Uniroyal-Elec-0805W8F1002T5E_C17414.pdf" H 3000 3350 50  0001 C CNN
+F 4 "C17414" H 3000 3350 50  0001 C CNN "LCSC"
+F 5 "0805W8F1000T5E" H 3000 3350 50  0001 C CNN "Mfc"
 	1    3000 3350
 	1    0    0    -1
@@
 P 3000 5350
 F 0 "R18" H 3070 5396 50  0000 L CNN
-F 1 "10K" H 3070 5305 50  0000 L CNN
+F 1 "10kOhm" H 3070 5305 50  0000 L CNN
 F 2 "" V 2930 5350 50  0001 C CNN
-F 3 "~" H 3000 5350 50  0001 C CNN
+F 3 "https://datasheet.lcsc.com/szlcsc/1810271610_UNI-ROYAL-Uniroyal-Elec-0805W8F1002T5E_C17414.pdf" H 3000 5350 50  0001 C CNN
+F 4 "C17414" H 3000 5350 50  0001 C CNN "LCSC"
+F 5 "0805W8F1000T5E" H 3000 5350 50  0001 C CNN "Mfc"
 	1    3000 5350
 	1    0    0    -1
@@
 P 5000 5350
 F 0 "R22" H 5070 5396 50  0000 L CNN
-F 1 "10K" H 5070 5305 50  0000 L CNN
+F 1 "10kOhm" H 5070 5305 50  0000 L CNN
 F 2 "" V 4930 5350 50  0001 C CNN
-F 3 "~" H 5000 5350 50  0001 C CNN
+F 3 "https://datasheet.lcsc.com/szlcsc/1810271610_UNI-ROYAL-Uniroyal-Elec-0805W8F1002T5E_C17414.pdf" H 5000 5350 50  0001 C CNN
+F 4 "C17414" H 5000 5350 50  0001 C CNN "LCSC"
+F 5 "0805W8F1000T5E" H 5000 5350 50  0001 C CNN "Mfc"
 	1    5000 5350
 	1    0    0    -1
@@
 P 3000 4350
 F 0 "R17" H 3070 4396 50  0000 L CNN
-F 1 "10K" H 3070 4305 50  0000 L CNN
+F 1 "10kOhm" H 3070 4305 50  0000 L CNN
 F 2 "" V 2930 4350 50  0001 C CNN
-F 3 "~" H 3000 4350 50  0001 C CNN
+F 3 "https://datasheet.lcsc.com/szlcsc/1810271610_UNI-ROYAL-Uniroyal-Elec-0805W8F1002T5E_C17414.pdf" H 3000 4350 50  0001 C CNN
+F 4 "C17414" H 3000 4350 50  0001 C CNN "LCSC"
+F 5 "0805W8F1000T5E" H 3000 4350 50  0001 C CNN "Mfc"
 	1    3000 4350
 	1    0    0    -1
@@
 P 5000 4350
 F 0 "R21" H 5070 4396 50  0000 L CNN
-F 1 "10K" H 5070 4305 50  0000 L CNN
+F 1 "10kOhm" H 5070 4305 50  0000 L CNN
 F 2 "" V 4930 4350 50  0001 C CNN
-F 3 "~" H 5000 4350 50  0001 C CNN
+F 3 "https://datasheet.lcsc.com/szlcsc/1810271610_UNI-ROYAL-Uniroyal-Elec-0805W8F1002T5E_C17414.pdf" H 5000 4350 50  0001 C CNN
+F 4 "C17414" H 5000 4350 50  0001 C CNN "LCSC"
+F 5 "0805W8F1000T5E" H 5000 4350 50  0001 C CNN "Mfc"
 	1    5000 4350
 	1    0    0    -1
@@
 P 5000 2350
 F 0 "R19" H 5070 2396 50  0000 L CNN
-F 1 "10K" H 5070 2305 50  0000 L CNN
+F 1 "10kOhm" H 5070 2305 50  0000 L CNN
 F 2 "" V 4930 2350 50  0001 C CNN
-F 3 "~" H 5000 2350 50  0001 C CNN
+F 3 "https://datasheet.lcsc.com/szlcsc/1810271610_UNI-ROYAL-Uniroyal-Elec-0805W8F1002T5E_C17414.pdf" H 5000 2350 50  0001 C CNN
+F 4 "C17414" H 5000 2350 50  0001 C CNN "LCSC"
+F 5 "0805W8F1000T5E" H 5000 2350 50  0001 C CNN "Mfc"
 	1    5000 2350
 	1    0    0    -1
@@
 P 5000 3350
 F 0 "R20" H 5070 3396 50  0000 L CNN
-F 1 "10K" H 5070 3305 50  0000 L CNN
+F 1 "10kOhm" H 5070 3305 50  0000 L CNN
 F 2 "" V 4930 3350 50  0001 C CNN
-F 3 "~" H 5000 3350 50  0001 C CNN
+F 3 "https://datasheet.lcsc.com/szlcsc/1810271610_UNI-ROYAL-Uniroyal-Elec-0805W8F1002T5E_C17414.pdf" H 5000 3350 50  0001 C CNN
+F 4 "C17414" H 5000 3350 50  0001 C CNN "LCSC"
+F 5 "0805W8F1000T5E" H 5000 3350 50  0001 C CNN "Mfc"
 	1    5000 3350
 	1    0    0    -1
@@
 Connection ~ 3000 2500
 Wire Wire Line
-	3000 2200 3000 2100
-Wire Wire Line
 	4000 2200 4000 2100
 Wire Wire Line
@@
 	3000 5200 3000 5100
 Wire Wire Line
-	4000 5100 4000 5200
-Wire Wire Line
 	4200 5500 5000 5500
 Connection ~ 5000 5500
@@
 Wire Wire Line
 	5000 5200 5000 5100
+Wire Wire Line
+	4000 5200 4000 5100
+Wire Wire Line
+	3000 2200 3000 2100
 $EndSCHEMATC

Commit message: Done PCB Sch Work
Parts:
- R15, R16, R17, R18, R19, R20, R21, R22: footprint (none) -> Resistor_SMD:R_0805_2012Metric_Pad1.15x1.40mm_HandSolder; Mfc 0805W8F1000T5E -> 0805W8F1002T5E
Changed lines of the file:
@@
 F 0 "R15" H 3070 2396 50  0000 L CNN
 F 1 "10kOhm" H 3070 2305 50  0000 L CNN
-F 2 "" V 2930 2350 50  0001 C CNN
+F 2 "Resistor_SMD:R_0805_2012Metric_Pad1.15x1.40mm_HandSolder" V 2930 2350 50  0001 C CNN
 F 3 "https://datasheet.lcsc.com/szlcsc/1810271610_UNI-ROYAL-Uniroyal-Elec-0805W8F1002T5E_C17414.pdf" H 3000 2350 50  0001 C CNN
 F 4 "C17414" H 3000 2350 50  0001 C CNN "LCSC"
-F 5 "0805W8F1000T5E" H 3000 2350 50  0001 C CNN "Mfc"
+F 5 "0805W8F1002T5E" H 3000 2350 50  0001 C CNN "Mfc"
 	1    3000 2350
 	1    0    0    -1
@@
 F 0 "R16" H 3070 3396 50  0000 L CNN
 F 1 "10kOhm" H 3070 3305 50  0000 L CNN
-F 2 "" V 2930 3350 50  0001 C CNN
+F 2 "Resistor_SMD:R_0805_2012Metric_Pad1.15x1.40mm_HandSolder" V 2930 3350 50  0001 C CNN
 F 3 "https://datasheet.lcsc.com/szlcsc/1810271610_UNI-ROYAL-Uniroyal-Elec-0805W8F1002T5E_C17414.pdf" H 3000 3350 50  0001 C CNN
 F 4 "C17414" H 3000 3350 50  0001 C CNN "LCSC"
-F 5 "0805W8F1000T5E" H 3000 3350 50  0001 C CNN "Mfc"
+F 5 "0805W8F1002T5E" H 3000 3350 50  0001 C CNN "Mfc"
 	1    3000 3350
 	1    0    0    -1
@@
 F 0 "R18" H 3070 5396 50  0000 L CNN
 F 1 "10kOhm" H 3070 5305 50  0000 L CNN
-F 2 "" V 2930 5350 50  0001 C CNN
+F 2 "Resistor_SMD:R_0805_2012Metric_Pad1.15x1.40mm_HandSolder" V 2930 5350 50  0001 C CNN
 F 3 "https://datasheet.lcsc.com/szlcsc/1810271610_UNI-ROYAL-Uniroyal-Elec-0805W8F1002T5E_C17414.pdf" H 3000 5350 50  0001 C CNN
 F 4 "C17414" H 3000 5350 50  0001 C CNN "LCSC"
-F 5 "0805W8F1000T5E" H 3000 5350 50  0001 C CNN "Mfc"
+F 5 "0805W8F1002T5E" H 3000 5350 50  0001 C CNN "Mfc"
 	1    3000 5350
 	1    0    0    -1
@@
 F 0 "R22" H 5070 5396 50  0000 L CNN
 F 1 "10kOhm" H 5070 5305 50  0000 L CNN
-F 2 "" V 4930 5350 50  0001 C CNN
+F 2 "Resistor_SMD:R_0805_2012Metric_Pad1.15x1.40mm_HandSolder" V 4930 5350 50  0001 C CNN
 F 3 "https://datasheet.lcsc.com/szlcsc/1810271610_UNI-ROYAL-Uniroyal-Elec-0805W8F1002T5E_C17414.pdf" H 5000 5350 50  0001 C CNN
 F 4 "C17414" H 5000 5350 50  0001 C CNN "LCSC"
-F 5 "0805W8F1000T5E" H 5000 5350 50  0001 C CNN "Mfc"
+F 5 "0805W8F1002T5E" H 5000 5350 50  0001 C CNN "Mfc"
 	1    5000 5350
 	1    0    0    -1
@@
 F 0 "R17" H 3070 4396 50  0000 L CNN
 F 1 "10kOhm" H 3070 4305 50  0000 L CNN
-F 2 "" V 2930 4350 50  0001 C CNN
+F 2 "Resistor_SMD:R_0805_2012Metric_Pad1.15x1.40mm_HandSolder" V 2930 4350 50  0001 C CNN
 F 3 "https://datasheet.lcsc.com/szlcsc/1810271610_UNI-ROYAL-Uniroyal-Elec-0805W8F1002T5E_C17414.pdf" H 3000 4350 50  0001 C CNN
 F 4 "C17414" H 3000 4350 50  0001 C CNN "LCSC"
-F 5 "0805W8F1000T5E" H 3000 4350 50  0001 C CNN "Mfc"
+F 5 "0805W8F1002T5E" H 3000 4350 50  0001 C CNN "Mfc"
 	1    3000 4350
 	1    0    0    -1
@@
 F 0 "R21" H 5070 4396 50  0000 L CNN
 F 1 "10kOhm" H 5070 4305 50  0000 L CNN
-F 2 "" V 4930 4350 50  0001 C CNN
+F 2 "Resistor_SMD:R_0805_2012Metric_Pad1.15x1.40mm_HandSolder" V 4930 4350 50  0001 C CNN
 F 3 "https://datasheet.lcsc.com/szlcsc/1810271610_UNI-ROYAL-Uniroyal-Elec-0805W8F1002T5E_C17414.pdf" H 5000 4350 50  0001 C CNN
 F 4 "C17414" H 5000 4350 50  0001 C CNN "LCSC"
-F 5 "0805W8F1000T5E" H 5000 4350 50  0001 C CNN "Mfc"
+F 5 "0805W8F1002T5E" H 5000 4350 50  0001 C CNN "Mfc"
 	1    5000 4350
 	1    0    0    -1
@@
 F 0 "R19" H 5070 2396 50  0000 L CNN
 F 1 "10kOhm" H 5070 2305 50  0000 L CNN
-F 2 "" V 4930 2350 50  0001 C CNN
+F 2 "Resistor_SMD:R_0805_2012Metric_Pad1.15x1.40mm_HandSolder" V 4930 2350 50  0001 C CNN
 F 3 "https://datasheet.lcsc.com/szlcsc/1810271610_UNI-ROYAL-Uniroyal-Elec-0805W8F1002T5E_C17414.pdf" H 5000 2350 50  0001 C CNN
 F 4 "C17414" H 5000 2350 50  0001 C CNN "LCSC"
-F 5 "0805W8F1000T5E" H 5000 2350 50  0001 C CNN "Mfc"
+F 5 "0805W8F1002T5E" H 5000 2350 50  0001 C CNN "Mfc"
 	1    5000 2350
 	1    0    0    -1
@@
 F 0 "R20" H 5070 3396 50  0000 L CNN
 F 1 "10kOhm" H 5070 3305 50  0000 L CNN
-F 2 "" V 4930 3350 50  0001 C CNN
+F 2 "Resistor_SMD:R_0805_2012Metric_Pad1.15x1.40mm_HandSolder" V 4930 3350 50  0001 C CNN
 F 3 "https://datasheet.lcsc.com/szlcsc/1810271610_UNI-ROYAL-Uniroyal-Elec-0805W8F1002T5E_C17414.pdf" H 5000 3350 50  0001 C CNN
 F 4 "C17414" H 5000 3350 50  0001 C CNN "LCSC"
-F 5 "0805W8F1000T5E" H 5000 3350 50  0001 C CNN "Mfc"
+F 5 "0805W8F1002T5E" H 5000 3350 50  0001 C CNN "Mfc"
 	1    5000 3350
 	1    0    0    -1
