File: Brewnode_PCB/MCU_Connector.sch (KiCad schematic (older format))
At the start: 1 part

Commit message: More PCB Sch work
Parts:
- removed J?: Conn_01x14, symbol Connector_Generic:Conn_01x14
- added J17: THD0510-16CL-GF, symbol Connector_Generic:Conn_01x16
Connections:
- wire segments 33 -> 39
Changed lines of the file:
@@
 3V3_ADC_Int
 $Comp
-L Connector_Generic:Conn_01x14 J?
-U 1 1 5F61BE26
-P 5500 3500
-F 0 "J?" H 5418 2575 50  0000 C CNN
-F 1 "Conn_01x14" H 5418 2666 50  0000 C CNN
-F 2 "" H 5500 3500 50  0001 C CNN
-F 3 "~" H 5500 3500 50  0001 C CNN
-	1    5500 3500
+L Connector_Generic:Conn_01x16 J17
+U 1 1 5F62AB42
+P 6250 3700
+F 0 "J17" H 6168 2675 50  0000 C CNN
+F 1 "THD0510-16CL-GF" H 6168 2766 50  0000 C CNN
+F 2 "" H 6250 3700 50  0001 C CNN
+F 3 "~" H 6250 3700 50  0001 C CNN
+F 4 "C283123" H 6250 3700 50  0001 C CNN "LCSC"
+	1    6250 3700
 	-1   0    0    1
 $EndComp
 Wire Wire Line
-	5700 4100 7500 4100
+	9500 6000 7600 6000
 Wire Wire Line
-	7500 4100 7500 6000
+	7600 6000 7600 4400
 Wire Wire Line
-	7500 6000 9500 6000
+	7600 4400 6450 4400
 Wire Wire Line
-	5700 4000 7600 4000
+	6450 4300 7600 4300
 Wire Wire Line
-	7600 4000 7600 5500
+	7600 4300 7600 4400
+Connection ~ 7600 4400
 Wire Wire Line
-	7600 5500 9500 5500
+	9500 5500 7700 5500
 Wire Wire Line
-	5700 3900 7700 3900
+	9500 5000 7800 5000
 Wire Wire Line
-	7700 3900 7700 5000
+	9500 4500 7900 4500
 Wire Wire Line
-	7700 5000 9500 5000
+	9500 4000 8000 4000
 Wire Wire Line
-	5700 3800 7800 3800
+	6450 4200 7600 4200
 Wire Wire Line
-	7800 3800 7800 4500
+	7600 4200 7600 4300
+Connection ~ 7600 4300
 Wire Wire Line
-	7800 4500 9500 4500
+	7800 3800 6450 3800
 Wire Wire Line
-	5700 3700 7900 3700
+	7800 3800 7800 5000
 Wire Wire Line
-	7900 3700 7900 4000
+	7900 3700 6450 3700
 Wire Wire Line
-	7900 4000 9500 4000
+	7900 3700 7900 4500
 Wire Wire Line
-	5700 3600 7900 3600
+	8000 4000 8000 3600
 Wire Wire Line
-	7900 3600 7900 3500
+	8000 3600 6450 3600
 Wire Wire Line
-	7900 3500 9500 3500
+	9500 3500 6450 3500
 Wire Wire Line
-	5700 3500 7800 3500
+	9500 3000 8000 3000
 Wire Wire Line
-	7800 3500 7800 3000
+	8000 3000 8000 3400
 Wire Wire Line
-	7800 3000 9500 3000
+	8000 3400 6450 3400
 Wire Wire Line
-	5700 3400 7700 3400
+	9500 2500 7900 2500
 Wire Wire Line
-	7700 3400 7700 2500
+	7900 2500 7900 3300
 Wire Wire Line
-	7700 2500 9500 2500
+	7900 3300 6450 3300
 Wire Wire Line
-	5700 3300 7600 3300
+	9500 2000 7800 2000
 Wire Wire Line
-	7600 3300 7600 2000
+	7800 2000 7800 3200
 Wire Wire Line
-	7600 2000 9500 2000
+	7800 3200 6450 3200
 Wire Wire Line
-	5700 3200 7500 3200
+	9500 1500 7700 1500
 Wire Wire Line
-	7500 3200 7500 1500
+	7700 1500 7700 3100
 Wire Wire Line
-	7500 1500 9500 1500
+	7700 3100 6450 3100
 Wire Wire Line
-	9500 1000 7400 1000
+	9500 1000 7600 1000
 Wire Wire Line
-	7400 1000 7400 3100
+	7600 1000 7600 3000
 Wire Wire Line
-	7400 3100 5700 3100
+	7600 3000 6450 3000
+Wire Wire Line
+	7700 3900 7700 4000
+Wire Wire Line
+	6450 3900 7700 3900
+Wire Wire Line
+	6450 4000 7700 4000
+Connection ~ 7700 4000
+Wire Wire Line
+	7700 4000 7700 4100
+Wire Wire Line
+	6450 4100 7700 4100
+Connection ~ 7700 4100
+Wire Wire Line
+	7700 4100 7700 5500
 $EndSCHEMATC

Commit message: More PCB Sch work
Parts:
- J17: value THD0510-16CL-GF -> 16p FPC; Mfc (none) -> THD0510-16CL-GF
Connections:
- no-connect marks 0 -> 1
Changed lines of the file:
@@
 P 6250 3700
 F 0 "J17" H 6168 2675 50  0000 C CNN
-F 1 "THD0510-16CL-GF" H 6168 2766 50  0000 C CNN
+F 1 "16p FPC" H 6168 2766 50  0000 C CNN
 F 2 "" H 6250 3700 50  0001 C CNN
-F 3 "~" H 6250 3700 50  0001 C CNN
+F 3 "https://datasheet.lcsc.com/szlcsc/1811021340_THD-THD0510-16CL-GF_C283123.pdf" H 6250 3700 50  0001 C CNN
 F 4 "C283123" H 6250 3700 50  0001 C CNN "LCSC"
+F 5 "THD0510-16CL-GF" H 6250 3700 50  0001 C CNN "Mfc"
 	1    6250 3700
 	-1   0    0    1
 $EndComp
-Wire Wire Line
-	9500 6000 7600 6000
 Wire Wire Line
 	7600 6000 7600 4400
@@
 	7600 4300 7600 4400
 Connection ~ 7600 4400
-Wire Wire Line
-	9500 5500 7700 5500
-Wire Wire Line
-	9500 5000 7800 5000
 Wire Wire Line
 	9500 4500 7900 4500
@@
 Wire Wire Line
 	7700 4100 7700 5500
+NoConn ~ 6450 2900
+Wire Wire Line
+	7800 5000 9500 5000
+Wire Wire Line
+	7700 5500 9500 5500
+Wire Wire Line
+	7600 6000 9500 6000
 $EndSCHEMATC

Commit message: Done PCB Sch Work
Parts:
- J17: footprint (none) -> Connector_FFC-FPC:Hirose_FH34_FPC_16; LCSC C283123 -> C324725; Mfc THD0510-16CL-GF -> FH34SRJ-16S-0.5SH(50)
Changed lines of the file:
@@
 F 0 "J17" H 6168 2675 50  0000 C CNN
 F 1 "16p FPC" H 6168 2766 50  0000 C CNN
-F 2 "" H 6250 3700 50  0001 C CNN
-F 3 "https://datasheet.lcsc.com/szlcsc/1811021340_THD-THD0510-16CL-GF_C283123.pdf" H 6250 3700 50  0001 C CNN
-F 4 "C283123" H 6250 3700 50  0001 C CNN "LCSC"
-F 5 "THD0510-16CL-GF" H 6250 3700 50  0001 C CNN "Mfc"
+F 2 "Connector_FFC-FPC:Hirose_FH34_FPC_16" H 6250 3700 50  0001 C CNN
+F 3 "https://datasheet.lcsc.com/szlcsc/1811071030_HRS-Hirose-FH34SRJ-16S-0-5SH-50_C324725.pdf" H 6250 3700 50  0001 C CNN
+F 4 "C324725" H 6250 3700 50  0001 C CNN "LCSC"
+F 5 "FH34SRJ-16S-0.5SH(50)" H 6250 3700 50  0001 C CNN "Mfc"
 	1    6250 3700
 	-1   0    0    1

Commit message: PCB Corrected library
Parts:
- J17: footprint Connector_FFC-FPC:Hirose_FH34_FPC_16 -> Tobbe_Hirose:Hirose_FH34_FPC_16
Changed lines of the file:
@@
 F 0 "J17" H 6168 2675 50  0000 C CNN
 F 1 "16p FPC" H 6168 2766 50  0000 C CNN
-F 2 "Connector_FFC-FPC:Hirose_FH34_FPC_16" H 6250 3700 50  0001 C CNN
+F 2 "Tobbe_Hirose:Hirose_FH34_FPC_16" H 6250 3700 50  0001 C CNN
 F 3 "https://datasheet.lcsc.com/szlcsc/1811071030_HRS-Hirose-FH34SRJ-16S-0-5SH-50_C324725.pdf" H 6250 3700 50  0001 C CNN
 F 4 "C324725" H 6250 3700 50  0001 C CNN "LCSC"
